Commit message: DIMESNIONS CONMPLETED

File: robot.xacro (robot description, xacro)
@@ -19,3 +19,12 @@
     value ="0.1"/>
 <!-- other dimensions -->
+ <xacro:property name = "s1"
+    value = "${body_height/2 + radius}"/>
+ <xacro:property name = "s2"
+ value ="${radius*2}"/>
+ <xacro:property name = name "s3"
+    value = "${radius*2}"/>
+ <xacro:property name = "s4"
+ value ="${body_width/2 + width/2}"/>
+<!-- MASS NAD INERTIA -->
 </robot>

Commit message: Mass added

File: robot.xacro (robot description, xacro)
@@ -13,8 +13,8 @@
 <!-- WHEEL DIMENSIONS  AND CASTOR DIMENSIONS -->
 <!-- RADIUS -->
-  <xacro:property name = "radius"
+<xacro:property name = "radius"
     value = "0.15"/>
 <! -- WIDTH  WHEEL -- >
-    <xacro:property name ="width"
+<xacro:property name ="width"
     value ="0.1"/>
 <!-- other dimensions -->
@@ -26,5 +26,25 @@
     value = "${radius*2}"/>
  <xacro:property name = "s4"
- value ="${body_width/2 + width/2}"/>
+   value ="${body_width/2 + width/2}"/>
 <!-- MASS NAD INERTIA -->
+<!-- DENSITY -->
+<!-- BODY LINK -->
+<xacro:macro name = "body_link"
+   value = "2710.0"/>
+<!-- WHEEL LINK -->
+<xacro:property name = "wheel_link"
+   value = "2710.0"/>
+<!-- CASTOR LINK -->
+<xacro:property name = "castor_link"
+   value = "2710.0"/>
+<!-- MASS -->
+<!-- BODY LINK MASS -->
+<xacro:property name = "body_mass"
+   value = "${body_linkk*body_length*body_width*body_height}"/>
+<!-- WHEEL LINK MASS -->
+<xacro:property name = "wheel_mass"
+   value = "${wheel_link*pi_const^2*radius*width}"/>
+<!-- CASTOR LINK MASS -->
+<xacro:property name = "castor_mass"
+   value = "${castor_link*1.3333*pi_const*radius^3}"/>
 </robot>

Commit message: moment of inertia added

File: robot.xacro (robot description, xacro)
@@ -7,7 +7,7 @@
  <xacro:property name = "body_length"
     value ="1"/>
+ <xacro:property name = "body_height"
+    value ="0.6"/>
  <xacro:property name = "body_width"
-    value ="0.6"/>
- <xacro:property name = "body_height"
     value ="0.3"/>
 <!-- WHEEL DIMENSIONS  AND CASTOR DIMENSIONS -->
@@ -47,4 +47,26 @@
 <!-- CASTOR LINK MASS -->
 <xacro:property name = "castor_mass"
-   value = "${castor_link*1.3333*pi_const*radius^3}"/>
+   value = "${castor_link*(4/3)*pi_const*radius^3}"/>
+<!--MOMENT OF INERTIA -->
+<!-- BODY LINK MOMENT OF INERTIA -->
+<xacro:property name = "Ix_body"
+   value = "${(1/12)*body_mass*(body_height^2 + body_width^2)}" />
+<xacro:property name = "Iy_body"
+   value = "${(1/12)*body_mass*(body_length^2 + body_width^2)}" />
+<xacro:property name = "Iz_body"
+   value = "${(1/12)*body_mass*(body_length^2 + body_height^2)}" />
+<!-- WHEEL LINK MOMENT OF INERTIA -->
+<xacro:property name = "Ix_wheel"
+   value = "${(1/12*wheel_mass)*(3*radius^2 + width^2)}" />
+<xacro:property name = "Iy_wheel"
+   value = "${(1/12)*wheel_mass*(radius^2 + width^2)}" />
+<xacro:property name = "Iz_wheel"
+   value = "${(1/2)*wheel_mass*radius^2}" />
+<!-- CASTOR LINK MOMENT OF INERTIA -->
+<xacro:property name = "Ix_castor"
+   value = "${(2/5)*castor_mass*radius^3}" />
+<xacro:property name = "Iy_castor"
+   value = "${(2/5)*castor_mass*radius^3}" />
+<xacro:property name = "Iz_castor"
+   value = "${(2/5)*castor_mass*radius^3}" />
 </robot>

Commit message: Inertia defined

File: robot.xacro (robot description, xacro)
@@ -5,25 +5,25 @@
 <!-- BODY LINK DIMENSIONS  -->
 <!-- units used in meters -->
- <xacro:property name = "body_length"
-    value ="1"/>
- <xacro:property name = "body_height"
-    value ="0.6"/>
- <xacro:property name = "body_width"
-    value ="0.3"/>
+<xacro:property name = "body_length"
+   value ="1"/>
+<xacro:property name = "body_height"
+   value ="0.6"/>
+<xacro:property name = "body_width"
+   value ="0.3"/>
 <!-- WHEEL DIMENSIONS  AND CASTOR DIMENSIONS -->
 <!-- RADIUS -->
 <xacro:property name = "radius"
-    value = "0.15"/>
-<! -- WIDTH  WHEEL -- >
+   value = "0.15"/>
+<!-- WIDTH  WHEEL -->
 <xacro:property name ="width"
-    value ="0.1"/>
+   value ="0.1"/>
 <!-- other dimensions -->
- <xacro:property name = "s1"
-    value = "${body_height/2 + radius}"/>
- <xacro:property name = "s2"
- value ="${radius*2}"/>
- <xacro:property name = name "s3"
-    value = "${radius*2}"/>
- <xacro:property name = "s4"
+<xacro:property name = "s1"
+   value = "${body_height/2 + radius}"/>
+<xacro:property name = "s2"
+   value ="${radius*2}"/>
+<xacro:property name = "s3"
+   value = "${radius*2}"/>
+<xacro:property name = "s4"
    value ="${body_width/2 + width/2}"/>
 <!-- MASS NAD INERTIA -->
@@ -65,8 +65,36 @@
 <!-- CASTOR LINK MOMENT OF INERTIA -->
 <xacro:property name = "Ix_castor"
-   value = "${(2/5)*castor_mass*radius*radius*radius}" />
+   value = "${(2/5)*castor_mass*radius*radius}" />
 <xacro:property name = "Iy_castor"
-   value = "${(2/5)*castor_mass*radius*radius*radius}" />
+   value = "${(2/5)*castor_mass*radius*radius}" />
 <xacro:property name = "Iz_castor"
-   value = "${(2/5)*castor_mass*radius*radius*radius}" />
+   value = "${(2/5)*castor_mass*radius*radius}" />
+<!-- complete inertial system of the body -->
+<!-- THE BASIC COORDINATE SYSTEM IS CENTERED AT THE GEOMETRIC CENTER OF THE BODY LINK -->
+<!-- BODY LINK -->
+<xacro:macro name = "body_link_macro">
+   <inertial>
+   <origin xyz = " 0 0 ${s1}" rpy = "0 0 0"/>
+   <mass value = "${body_mass}"/>
+   <inertia ixx ="${Ix_body}" ixy = "0.0" ixz ="0.0" iyy ="${Iy_body}" iyz = "0.0" izz= "${Iz_body}"/>
+   </inertial>
+</xacro:macro>
+<!-- WHEEL LINK -->
+<xacro:macro name = "wheel_link_macro">
+   <inertial>
+   <origin xyz = "0 0 0" rpy = " 1.570795 0 0"/>
+   <mass value = "${wheel_mass}"/>
+   <inertia ixx ="${Ix_wheel}" ixy="0.0" ixz="0.0" iyy="${Iy_wheel}" iyz ="0.0" izz="${Iz_wheel}"/>
+   </inertial>
+</xacro:macro>
+<!-- CASTOR LINK -->
+<xacro:macro name = "castor_link_macro">
+   <inertial>
+   <origin xyz = "0 0 0" rpy = "0 0 0"/>
+   <mass value = "${castor_mass}"/>
+   <inertia ixx = "${Ix_castor}" ixy= "0.0" ixz="0.0" iyy="${Iy_castor}" iyz="0.0" izz= "${Iz_castor}"/>
+   </inertial>
+</xacro:macro>
+<!-- INERTFACE FOR COMTROLS -->
+<!-- DEFINING LINKS ANDS JOINTS -->
 </robot>

Commit message: main body joint

File: robot.xacro (robot description, xacro)
@@ -97,4 +97,26 @@
 </xacro:macro>
 <!-- INERTFACE FOR COMTROLS -->
+<!-- FICTOUS LINK  -->
 <!-- DEFINING LINKS ANDS JOINTS -->
+<link name  = "body_footprint"></link>
+<joint name "body_link_joint" type = "fixed">
+   <parent link = " base_footprint "/>
+   <child link = "body_link"/>
+</joint>
+<!-- BODY LINK OF ROBOT -->
+<link name = "body_link">
+   <visual>
+      <geometry>
+         <box size = "${body_length} ${body_width} ${body_height}"/>
+      </geometry>
+      <origin xyz="0 0 ${s1}" rpy = "0 0 0"/>
+   </visual>
+   <collison>
+      <geometry>
+         <box size = "${body_length} ${body_width} ${body_height}"/>
+      </geometry>
+      <origin xyz="0 0 ${s1}" rpy = "0 0 0"/>
+   </collison>
+   <xacro:inertia_body_macro/>
+</link>
 </robot>

Commit message: wheel joints added

File: robot.xacro (robot description, xacro)
@@ -120,3 +120,50 @@
    <xacro:inertia_body_macro/>
 </link>
+<!-- WHEEL JOINT -->
+<joint name="wheel1_joint" type ="continuous">
+   <parent link = "body_link"/>
+   <child link = "wheel1_link"/>
+   <origin xyz= " ${-s2} ${-s4} {r}" rpy="0 0 0"/>
+   <axis xyz= "0 1 0"/>
+   <limit effort = "100000" velocity= "10"/>
+   <dyanmic damping ="1.0" friction ="1.0"/>
+</joint>
+<link name = "wheel1_link">
+   <visaul>
+      <geometry>
+         <cylinder length = "${width}" radius = "${radius}"/>
+      </geometry>
+      <origin xyz = "0 0 0" rpy = "1.570795 0 0"/>
+   </visual>
+   <collision>
+      <geometry>
+         <cylinder length = "${width}" radius = "${radius}"/>
+      </geometry>
+      <origin xyz = "0 0 0" rpy = "1.570795 0 0"/>
+   </collision>
+   <xacro:inertia_wheel_macro/>
+</link>
+<joint name="wheel2_joint" type ="continuous">
+   <parent link = "body_link"/>
+   <child link = "wheel2_link"/>
+   <origin xyz= " ${-s2} ${s4} {r}" rpy="0 0 0"/>
+   <axis xyz= "0 1 0"/>
+   <limit effort = "100000" velocity= "10"/>
+   <dyanmic damping ="1.0" friction ="1.0"/>
+</joint>
+<link name = "wheel2_link">
+   <visaul>
+      <geometry>
+         <cylinder length = "${width}" radius = "${radius}"/>
+      </geometry>
+      <origin xyz = "0 0 0" rpy = "1.570795 0 0"/>
+   </visual>
+   <collision>
+      <geometry>
+         <cylinder length = "${width}" radius = "${radius}"/>
+      </geometry>
+      <origin xyz = "0 0 0" rpy = "1.570795 0 0"/>
+   </collision>
+   <xacro:inertia_wheel_macro/>
+</link>
 </robot>
