Commit message: castor lionk added in xacro file

File: install/mobile_robot/share/mobile_robot/model/robot.xacro (robot description, xacro)
@@ -39,23 +39,17 @@
 <!-- BODY LINK MOMENT OF INERTIA -->
 <xacro:property name="Ix_body"
-   value="${(1/12)*body_mass*(body_height*body_height + body_width*body_width)}" />
+   value="${(1/12)*body_mass*(body_height*body_height + body_width*body_width)}"/>
 <xacro:property name="Iy_body"
-   value="${(1/12)*body_mass*(body_length*body_length + body_width*body_width)}" />
+   value="${(1/12)*body_mass*(body_length*body_length + body_width*body_width)}"/>
 <xacro:property name="Iz_body"
-   value="${(1/12)*body_mass*(body_length*body_length + body_height*body_height)}" />
+   value="${(1/12)*body_mass*(body_length*body_length + body_height*body_height)}"/>
 <!-- WHEEL LINK MOMENT OF INERTIA -->
-<xacro:property name="Ix_wheel"
-   value="${(1/12)*wheel_mass*(3*radius*radius + width*width)}" />
-<xacro:property name="Iy_wheel"
-   value="${(1/12)*wheel_mass*(radius*radius + width*width)}" />
-<xacro:property name="Iz_wheel"
-   value="${(1/2)*wheel_mass*radius*radius}" />
+<xacro:property name="Ix_wheel" value="0.01"/>
+<xacro:property name="Iy_wheel" value="0.01"/>
+<xacro:property name="Iz_wheel" value="0.01"/>
 <!-- CASTOR LINK MOMENT OF INERTIA -->
-<xacro:property name="Ix_castor"
-   value="${(2/5)*castor_mass*radius*radius}" />
-<xacro:property name="Iy_castor"
-   value="${(2/5)*castor_mass*radius*radius}" />
-<xacro:property name="Iz_castor"
-   value="${(2/5)*castor_mass*radius*radius}" />
+<xacro:property name="Ix_castor" value="0.005"/>
+<xacro:property name="Iy_castor" value="0.005"/>
+<xacro:property name="Iz_castor" value="0.005"/>
 <!-- complete inertial system of the body -->
 <!-- FILE THAT INCLUDES GAZEBO OPTIONS AND MOTION CONTROLS-->
@@ -64,31 +58,25 @@
 <!-- BODY LINK -->
 <xacro:macro name="body_link_macro">
-   <inertial>
-     <origin xyz="0 0 ${s1}" rpy="0 0 0"/>
-     <mass value="${body_mass}"/>
-     <inertia ixx="${Ix_body}" ixy="0.0" ixz="0.0"
-              iyy="${Iy_body}" iyz="0.0"
-              izz="${Iz_body}"/>
-   </inertial>
+  <inertial>
+    <origin xyz="0 0 ${s1}" rpy="0 0 0"/>
+    <mass value="${body_mass}"/>
+    <inertia ixx="1.0" ixy="0" ixz="0" iyy="1.0" iyz="0" izz="1.0"/>
+  </inertial>
 </xacro:macro>
 <!-- WHEEL LINK -->
 <xacro:macro name="wheel_link_macro">
-   <inertial>
-     <origin xyz="0 0 0" rpy="1.570795 0 0"/>
-     <mass value="${wheel_mass}"/>
-     <inertia ixx="${Ix_wheel}" ixy="0.0" ixz="0.0"
-              iyy="${Iy_wheel}" iyz="0.0"
-              izz="${Iz_wheel}"/>
-   </inertial>
+  <inertial>
+    <origin xyz="0 0 0" rpy="0 0 0"/>
+    <mass value="2.0"/>
+    <inertia ixx="0.01" ixy="0" ixz="0" iyy="0.01" iyz="0" izz="0.01"/>
+  </inertial>
 </xacro:macro>
 <!-- CASTOR LINK -->
 <xacro:macro name="castor_link_macro">
-   <inertial>
-     <origin xyz="0 0 0" rpy="0 0 0"/>
-     <mass value="${castor_mass}"/>
-     <inertia ixx="${Ix_castor}" ixy="0.0" ixz="0.0"
-              iyy="${Iy_castor}" iyz="0.0"
-              izz="${Iz_castor}"/>
-   </inertial>
+  <inertial>
+    <origin xyz="0 0 0" rpy="0 0 0"/>
+    <mass value="1.0"/>
+    <inertia ixx="0.005" ixy="0" ixz="0" iyy="0.005" iyz="0" izz="0.005"/>
+  </inertial>
 </xacro:macro>
 <!-- INERTFACE FOR COMTROLS -->
@@ -97,46 +85,85 @@
 <link name="body_footprint"/>
 <joint name="body_link_joint" type="fixed">
-   <parent link="body_footprint"/>
-   <child link="body_link"/>
+  <parent link="body_footprint"/>
+  <child link="body_link"/>
 </joint>
 <!-- BODY LINK OF ROBOT -->
 <link name="body_link">
-   <visual>
-      <geometry>
-         <box size="${body_length} ${body_width} ${body_height}"/>
-      </geometry>
-      <origin xyz="0 0 ${s1}" rpy="0 0 0"/>
-   </visual>
-   <collision>
-      <geometry>
-         <box size="${body_length} ${body_width} ${body_height}"/>
-      </geometry>
-      <origin xyz="0 0 ${s1}" rpy="0 0 0"/>
-   </collision>
-   <xacro:body_link_macro/>
+  <visual>
+    <geometry>
+      <box size="${body_length} ${body_width} ${body_height}"/>
+    </geometry>
+    <origin xyz="0 0 ${s1}" rpy="0 0 0"/>
+  </visual>
+  <collision>
+    <geometry>
+      <box size="${body_length} ${body_width} ${body_height}"/>
+    </geometry>
+    <origin xyz="0 0 ${s1}" rpy="0 0 0"/>
+  </collision>
+  <xacro:body_link_macro/>
 </link>
 <!-- WHEEL JOINT -->
 <joint name="wheel1_joint" type="continuous">
-   <parent link="body_link"/>
-   <child link="wheel1_link"/>
-   <origin xyz="${-s2} ${-s4} ${radius}" rpy="0 0 0"/>
-   <axis xyz="0 1 0"/>
-   <limit effort="100000" velocity="10"/>
-   <dynamics damping="1.0" friction="1.0"/>
+  <parent link="body_link"/>
+  <child link="wheel1_link"/>
+  <origin xyz="${-s2} ${-s4} ${radius}" rpy="0 0 0"/>
+  <axis xyz="0 1 0"/>
+  <dynamics damping="1.0" friction="1.0"/>
 </joint>
 <link name="wheel1_link">
-   <visual>
-      <geometry>
-         <cylinder length="${width}" radius="${radius}"/>
-      </geometry>
-      <origin xyz="0 0 0" rpy="1.570795 0 0"/>
-   </visual>
-   <collision>
-      <geometry>
-         <cylinder length="${width}" radius="${radius}"/>
-      </geometry>
-      <origin xyz="0 0 0" rpy="1.570795 0 0"/>
-   </collision>
-   <xacro:wheel_link_macro/>
+  <visual>
+    <geometry>
+      <cylinder length="${width}" radius="${radius}"/>
+    </geometry>
+    <origin xyz="0 0 0" rpy="1.570795 0 0"/>
+  </visual>
+  <collision>
+    <geometry>
+      <cylinder length="${width}" radius="${radius}"/>
+    </geometry>
+    <origin xyz="0 0 0" rpy="1.570795 0 0"/>
+  </collision>
+  <xacro:wheel_link_macro/>
+</link>
+<joint name="wheel2_joint" type="continuous">
+  <parent link="body_link"/>
+  <child link="wheel2_link"/>
+  <origin xyz="${-s2} ${s4} ${radius}" rpy="0 0 0"/>
+  <axis xyz="0 1 0"/>
+</joint>
+<link name="wheel2_link">
+  <visual>
+    <geometry>
+      <cylinder length="${width}" radius="${radius}"/>
+    </geometry>
+    <origin xyz="0 0 0" rpy="1.570795 0 0"/>
+  </visual>
+  <collision>
+    <geometry>
+      <cylinder length="${width}" radius="${radius}"/>
+    </geometry>
+    <origin xyz="0 0 0" rpy="1.570795 0 0"/>
+  </collision>
+  <xacro:wheel_link_macro/>
+</link>
+<!-- CASTOR WHEEL -->
+<joint name="castor_joint" type="fixed">
+  <parent link="body_link"/>
+  <child link="castor_link"/>
+  <origin xyz="${body_length/2} 0 ${radius/2}" rpy="0 0 0"/>
+</joint>
+<link name="castor_link">
+  <visual>
+    <geometry>
+      <sphere radius="${radius/2}"/>
+    </geometry>
+  </visual>
+  <collision>
+    <geometry>
+      <sphere radius="${radius/2}"/>
+    </geometry>
+  </collision>
+  <xacro:castor_link_macro/>
 </link>
 </robot>

File: src/mobile_robot/model/robot.xacro (robot description, xacro)
@@ -1,142 +1,195 @@
 <?xml version='1.0'?>
-<robot name="castor_robot" xmlns:xacro="http://www.ros.org/wiki/xacro">
+<robot name = "castor_robot" xmlns:xacro="http://www.ros.org/wiki/xacro">
 <!-- define constants -->
-<xacro:property name="ohm" value="3.14159"/>
+<xacro:property name = "ohm" value ="3.14159"/>
 <!-- BODY LINK DIMENSIONS  -->
 <!-- units used in meters -->
-<xacro:property name="body_length" value="1"/>
-<xacro:property name="body_height" value="0.6"/>
-<xacro:property name="body_width"  value="0.3"/>
+<xacro:property name = "body_length"
+   value ="1"/>
+<xacro:property name = "body_height"
+   value ="0.6"/>
+<xacro:property name = "body_width"
+   value ="0.3"/>
 <!-- WHEEL DIMENSIONS  AND CASTOR DIMENSIONS -->
 <!-- RADIUS -->
-<xacro:property name="radius" value="0.15"/>
+<xacro:property name = "radius"
+   value = "0.15"/>
 <!-- WIDTH  WHEEL -->
-<xacro:property name="width" value="0.1"/>
+<xacro:property name ="width"
+   value ="0.1"/>
 <!-- other dimensions -->
-<xacro:property name="s1" value="${body_height/2 + radius}"/>
-<xacro:property name="s2" value="${radius*2}"/>
-<xacro:property name="s3" value="${radius*2}"/>
-<xacro:property name="s4" value="${body_width/2 + width/2}"/>
+<xacro:property name = "s1"
+   value = "${body_height/2 + radius}"/>
+<xacro:property name = "s2"
+   value ="${radius*2}"/>
+<xacro:property name = "s3"
+   value = "${radius*2}"/>
+<xacro:property name = "s4"
+   value ="${body_width/2 + width/2}"/>
 <!-- MASS NAD INERTIA -->
 <!-- DENSITY -->
 <!-- BODY LINK -->
-<xacro:property name="body_link" value="2710.0"/>
+<xacro:property name = "body_link"
+   value = "2710.0"/>
 <!-- WHEEL LINK -->
-<xacro:property name="wheel_link" value="2710.0"/>
+<xacro:property name = "wheel_link"
+   value = "2710.0"/>
 <!-- CASTOR LINK -->
-<xacro:property name="castor_link" value="2710.0"/>
+<xacro:property name = "castor_link"
+   value = "2710.0"/>
 <!-- MASS -->
 <!-- BODY LINK MASS -->
-<xacro:property name="body_mass"
-   value="${body_link*body_length*body_width*body_height}"/>
+<xacro:property name = "body_mass"
+   value = "${body_link*body_length*body_width*body_height}"/>
 <!-- WHEEL LINK MASS -->
-<xacro:property name="wheel_mass"
-   value="${wheel_link*ohm*radius*radius*width}"/>
+<xacro:property name = "wheel_mass"
+   value = "${wheel_link*ohm*radius*radius*width}"/>
 <!-- CASTOR LINK MASS -->
-<xacro:property name="castor_mass"
-   value="${castor_link*(4/3)*ohm*radius*radius*radius}"/>
+<xacro:property name = "castor_mass"
+   value = "${castor_link*(4/3)*ohm*radius*radius*radius}"/>
 <!--MOMENT OF INERTIA -->
 <!-- BODY LINK MOMENT OF INERTIA -->
-<xacro:property name="Ix_body"
-   value="${(1/12)*body_mass*(body_height*body_height + body_width*body_width)}" />
-<xacro:property name="Iy_body"
-   value="${(1/12)*body_mass*(body_length*body_length + body_width*body_width)}" />
-<xacro:property name="Iz_body"
-   value="${(1/12)*body_mass*(body_length*body_length + body_height*body_height)}" />
+<xacro:property name = "Ix_body"
+   value = "${(1/12)*body_mass*(body_height*body_height + body_width*body_width)}" />
+<xacro:property name = "Iy_body"
+   value = "${(1/12)*body_mass*(body_length*body_length + body_width*body_width)}" />
+<xacro:property name = "Iz_body"
+   value = "${(1/12)*body_mass*(body_length*body_length + body_height*body_height)}" />
 <!-- WHEEL LINK MOMENT OF INERTIA -->
-<xacro:property name="Ix_wheel"
-   value="${(1/12)*wheel_mass*(3*radius*radius + width*width)}" />
-<xacro:property name="Iy_wheel"
-   value="${(1/12)*wheel_mass*(radius*radius + width*width)}" />
-<xacro:property name="Iz_wheel"
-   value="${(1/2)*wheel_mass*radius*radius}" />
+<xacro:property name = "Ix_wheel"
+   value = "${(1/12*wheel_mass)*(3*radius*radius + width*width)}" />
+<xacro:property name = "Iy_wheel"
+   value = "${(1/12)*wheel_mass*(radius*radius + width*width)}" />
+<xacro:property name = "Iz_wheel"
+   value = "${(1/2)*wheel_mass*radius*radius}" />
 <!-- CASTOR LINK MOMENT OF INERTIA -->
-<xacro:property name="Ix_castor"
-   value="${(2/5)*castor_mass*radius*radius}" />
-<xacro:property name="Iy_castor"
-   value="${(2/5)*castor_mass*radius*radius}" />
-<xacro:property name="Iz_castor"
-   value="${(2/5)*castor_mass*radius*radius}" />
+<xacro:property name = "Ix_castor"
+   value = "${(2/5)*castor_mass*radius*radius}" />
+<xacro:property name = "Iy_castor"
+   value = "${(2/5)*castor_mass*radius*radius}" />
+<xacro:property name = "Iz_castor"
+   value = "${(2/5)*castor_mass*radius*radius}" />
 <!-- complete inertial system of the body -->
 <!-- FILE THAT INCLUDES GAZEBO OPTIONS AND MOTION CONTROLS-->
-<xacro:include filename="$(find mobile_robot)/model/robot.gazebo"/>
+<xacro:include filename ="$(find mobile_robot)/model/robot.gazebo"/>
 <!-- THE BASIC COORDINATE SYSTEM IS CENTERED AT THE GEOMETRIC CENTER OF THE BODY LINK -->
 <!-- BODY LINK -->
-<xacro:macro name="body_link_macro">
+<xacro:macro name = "body_link_macro">
    <inertial>
-     <origin xyz="0 0 ${s1}" rpy="0 0 0"/>
-     <mass value="${body_mass}"/>
-     <inertia ixx="${Ix_body}" ixy="0.0" ixz="0.0"
-              iyy="${Iy_body}" iyz="0.0"
-              izz="${Iz_body}"/>
+   <origin xyz = " 0 0 ${s1}" rpy = "0 0 0"/>
+   <mass value = "${body_mass}"/>
+   <inertia ixx ="${Ix_body}" ixy = "0.0" ixz ="0.0" iyy ="${Iy_body}" iyz = "0.0" izz= "${Iz_body}"/>
    </inertial>
-</xacro:macro>
+</xacro:body_link_macro>
 <!-- WHEEL LINK -->
-<xacro:macro name="wheel_link_macro">
+<xacro:macro name = "wheel_link_macro">
    <inertial>
-     <origin xyz="0 0 0" rpy="1.570795 0 0"/>
-     <mass value="${wheel_mass}"/>
-     <inertia ixx="${Ix_wheel}" ixy="0.0" ixz="0.0"
-              iyy="${Iy_wheel}" iyz="0.0"
-              izz="${Iz_wheel}"/>
+   <origin xyz = "0 0 0" rpy = " 1.570795 0 0"/>
+   <mass value = "${wheel_mass}"/>
+   <inertia ixx ="${Ix_wheel}" ixy="0.0" ixz="0.0" iyy="${Iy_wheel}" iyz ="0.0" izz="${Iz_wheel}"/>
    </inertial>
-</xacro:macro>
+</xacro:wheel_link_macro>
 <!-- CASTOR LINK -->
-<xacro:macro name="castor_link_macro">
+<xacro:macro name = "castor_link_macro">
    <inertial>
-     <origin xyz="0 0 0" rpy="0 0 0"/>
-     <mass value="${castor_mass}"/>
-     <inertia ixx="${Ix_castor}" ixy="0.0" ixz="0.0"
-              iyy="${Iy_castor}" iyz="0.0"
-              izz="${Iz_castor}"/>
+   <origin xyz = "0 0 0" rpy = "0 0 0"/>
+   <mass value = "${castor_mass}"/>
+   <inertia ixx = "${Ix_castor}" ixy= "0.0" ixz="0.0" iyy="${Iy_castor}" iyz="0.0" izz= "${Iz_castor}"/>
    </inertial>
-</xacro:macro>
+</xacro:castor_link_macro>
 <!-- INERTFACE FOR COMTROLS -->
 <!-- FICTOUS LINK  -->
 <!-- DEFINING LINKS ANDS JOINTS -->
-<link name="body_footprint"/>
-<joint name="body_link_joint" type="fixed">
-   <parent link="body_footprint"/>
-   <child link="body_link"/>
+<link name  = "body_footprint"></link>
+<joint name = "body_link_joint" type = "fixed">
+   <parent link = " body_footprint "/>
+   <child link = "body_link"/>
 </joint>
 <!-- BODY LINK OF ROBOT -->
-<link name="body_link">
+<link name = "body_link">
    <visual>
       <geometry>
-         <box size="${body_length} ${body_width} ${body_height}"/>
+         <box size = "${body_length} ${body_width} ${body_height}"/>
       </geometry>
-      <origin xyz="0 0 ${s1}" rpy="0 0 0"/>
+      <origin xyz="0 0 ${s1}" rpy = "0 0 0"/>
    </visual>
    <collision>
       <geometry>
-         <box size="${body_length} ${body_width} ${body_height}"/>
+         <box size = "${body_length} ${body_width} ${body_height}"/>
       </geometry>
-      <origin xyz="0 0 ${s1}" rpy="0 0 0"/>
+      <origin xyz="0 0 ${s1}" rpy = "0 0 0"/>
    </collision>
    <xacro:body_link_macro/>
 </link>
 <!-- WHEEL JOINT -->
-<joint name="wheel1_joint" type="continuous">
-   <parent link="body_link"/>
-   <child link="wheel1_link"/>
-   <origin xyz="${-s2} ${-s4} ${radius}" rpy="0 0 0"/>
-   <axis xyz="0 1 0"/>
-   <limit effort="100000" velocity="10"/>
-   <dynamics damping="1.0" friction="1.0"/>
+<joint name="wheel1_joint" type ="continuous">
+   <parent link = "body_link"/>
+   <child link = "wheel1_link"/>
+   <origin xyz= " ${-s2} ${-s4} ${radius}" rpy="0 0 0"/>
+   <axis xyz= "0 1 0"/>
+   <limit effort = "100000" velocity= "10"/>
+   <dynamics damping ="1.0" friction ="1.0"/>
 </joint>
-<link name="wheel1_link">
+<link name = "wheel1_link">
    <visual>
       <geometry>
-         <cylinder length="${width}" radius="${radius}"/>
+         <cylinder length = "${width}" radius = "${radius}"/>
       </geometry>
-      <origin xyz="0 0 0" rpy="1.570795 0 0"/>
+      <origin xyz = "0 0 0" rpy = "1.570795 0 0"/>
    </visual>
    <collision>
       <geometry>
-         <cylinder length="${width}" radius="${radius}"/>
+         <cylinder length = "${width}" radius = "${radius}"/>
       </geometry>
-      <origin xyz="0 0 0" rpy="1.570795 0 0"/>
+      <origin xyz = "0 0 0" rpy = "1.570795 0 0"/>
    </collision>
    <xacro:wheel_link_macro/>
 </link>
+<joint name="wheel2_joint" type ="continuous">
+   <parent link = "body_link"/>
+   <child link = "wheel2_link"/>
+   <origin xyz= " ${-s2} ${s4} ${radius}" rpy="0 0 0"/>
+   <axis xyz= "0 1 0"/>
+   <limit effort = "100000" velocity= "10"/>
+   <dynamics damping ="1.0" friction ="1.0"/>
+</joint>
+<link name = "wheel2_link">
+   <visual>
+      <geometry>
+         <cylinder length = "${width}" radius = "${radius}"/>
+      </geometry>
+      <origin xyz = "0 0 0" rpy = "1.570795 0 0"/>
+   </visual>
+   <collision>
+      <geometry>
+         <cylinder length = "${width}" radius = "${radius}"/>
+      </geometry>
+      <origin xyz = "0 0 0" rpy = "1.570795 0 0"/>
+   </collision>
+   <xacro:wheel_link_macro/>
+</link>
+<!-- CASTOR JOINT -->
+<joint name="caster_joint" type ="continuous">
+   <parent link = "body_link"/>
+   <child link = "caster_link"/>
+   <origin xyz= " ${body_length/2 - radius} 0 ${radius}" rpy="0 0 0"/>
+   <axis xyz= "0 1 0"/>
+   <limit effort = "100000" velocity= "10"/>
+   <dynamics damping ="1.0" friction ="1.0"/>
+</joint>
+<link name = "caster_link">
+   <visual>
+      <geometry>
+         <sphere radius = "${radius}"/>
+      </geometry>
+      <origin xyz = "0 0 0" rpy = "0 0 0"/>
+   </visual>
+   <collision>
+      <geometry>
+         <sphere radius = "${radius}"/>
+      </geometry>
+      <origin xyz = "0 0 0" rpy = "0 0 0"/>
+   </collision>
+   <xacro:castor_link_macro/>
+</link>
 </robot>
