Commit message: latest change in.gazebo file

File: src/mobile_robot/model/robot.gazebo.xacro (robot description, xacro)
@@ -51,4 +51,9 @@
 <gazebo reference="lidar_link">
     <sensor name="gpu_lidar" type="gpu_ray">
+        <ray>
+            <collision>
+                <ignore_entity>castor_robot</ignore_entity>
+            </collision>
+        </ray>
     <pose relative_to="lidar_link">0 0 0 0 0 0</pose>
     <topic>/world/default/model/castor_robot/link/lidar_link/sensor/gpu_lidar/scan</topic>

Commit message: latest file

File: src/mobile_robot/model/robot.gazebo.xacro (robot description, xacro)
@@ -1,9 +1,9 @@
 <?xml version="1.0"?>
 <robot xmlns:xacro="https://www.ros.org/wiki/xacro">
-<gazebo>
+<!-- <gazebo>
     <model>
         <canonical_link>body_link</canonical_link>
     </model>
-</gazebo>
+</gazebo> -->
 <gazebo reference = "body_link">
     <mu1>0.2</mu1>

File: src/mobile_robot/model/robot.xacro (robot description, xacro)
@@ -207,10 +207,10 @@
       </geometry>
    </visual>
-   <collision name ="collision">
+   <!-- <collision name ="collision">
       <origin xyz="0 0 0" rpy="0 0 0"/>
       <geometry>
          <cylinder length ="0.1" radius="0.1"/>
       </geometry>
-   </collision>
+   </collision> -->
    <inertial>
       <mass value="1e-6"/>

Commit message: friction added for the all four wheels

File: src/mobile_robot/model/robot.gazebo.xacro (robot description, xacro)
@@ -21,9 +21,20 @@
     <material>Gazebo/Yellow</material>
 </gazebo>
-<gazebo reference = "caster_link">
+<gazebo reference = "wheel3_link">
+    <mu1>1.0</mu1>
+    <mu2>1.0</mu2>
+    <material>Gazebo/Yellow</material>
+</gazebo
+>
+<gazebo reference = "wheel4_link">
+    <mu1>1.0</mu1>
+    <mu2>1.0</mu2>
+    <material>Gazebo/Yellow</material>
+</gazebo>
+<!-- <gazebo reference = "caster_link">
     <mu1>0.00002</mu1>
     <mu2>0.00002</mu2>
     <material>Gazebo/Blue</material>
-</gazebo>
+</gazebo> -->
 <gazebo>
     <plugin filename = "libgz-sim-diff-drive-system.so" name="gz::sim::systems::DiffDrive">
