Commit message: dimensions updated

File: src/mobile_robot/model/robot.xacro (robot description, xacro)
@@ -6,16 +6,16 @@
 <!-- units used in meters -->
 <xacro:property name = "body_length"
-   value ="1.5"/>
+   value ="1.0"/>
+<xacro:property name = "body_width"
+   value ="0.3"/>
 <xacro:property name = "body_height"
-   value ="0.35"/>
-<xacro:property name = "body_width"
-   value ="0.55"/>
+   value ="0.6"/>
 <!-- WHEEL DIMENSIONS  AND CASTOR DIMENSIONS -->
 <!-- RADIUS -->
 <xacro:property name = "radius"
-   value = "0.18"/>
+   value = "0.15"/>
 <!-- WIDTH  WHEEL -->
 <xacro:property name ="width"
-   value ="0.12"/>
+   value ="0.1"/>
 <!-- other dimensions -->
 <xacro:property name = "s1"

Commit message: moment of inertia updated

File: src/mobile_robot/model/robot.xacro (robot description, xacro)
@@ -20,5 +20,5 @@
 <!-- other dimensions -->
 <xacro:property name = "s1"
-   value = "${body_height/2 + radius}"/>
+   value = "${body_width/2 + radius}"/>
 <xacro:property name = "s2"
    value ="${radius*2}"/>
@@ -26,26 +26,26 @@
    value = "${radius*2}"/>
 <xacro:property name = "s4"
-   value ="${body_width/2 + width/2}"/>
+   value ="${body_height/2 + width/2}"/>
 <!-- MASS NAD INERTIA -->
 <!-- DENSITY -->
 <!-- BODY LINK -->
-<xacro:property name = "body_link"
+<xacro:property name = "body"
    value = "2710.0"/>
 <!-- WHEEL LINK -->
-<xacro:property name = "wheel_link"
+<xacro:property name = "wheel"
    value = "2710.0"/>
 <!-- CASTOR LINK -->
-<xacro:property name = "castor_link"
+<xacro:property name = "castor"
    value = "2710.0"/>
 <!-- MASS -->
 <!-- BODY LINK MASS -->
 <xacro:property name = "body_mass"
-   value = "${body_link*body_length*body_width*body_height}"/>
+   value = "${body*body_length*body_width*body_height}"/>
 <!-- WHEEL LINK MASS -->
 <xacro:property name = "wheel_mass"
-   value = "${wheel_link*ohm*radius*radius*width}"/>
+   value = "${wheel*ohm*radius*radius*width}"/>
 <!-- CASTOR LINK MASS -->
 <xacro:property name = "castor_mass"
-   value = "${castor_link*(4/3)*ohm*radius*radius*radius}"/>
+   value = "${castor*(4.0/3.0)*ohm*radius*radius*radius}"/>
 <!--MOMENT OF INERTIA -->
 <!-- BODY LINK MOMENT OF INERTIA -->
@@ -58,16 +58,16 @@
 <!-- WHEEL LINK MOMENT OF INERTIA -->
 <xacro:property name="Ix_wheel"
-   value="${(1/12)*wheel_mass*(3*radius*radius + width*width)}"/>
+   value="${(1.0/12.0)*wheel_mass*(3*radius*radius + width*width)}"/>
 <xacro:property name="Iy_wheel"
-   value="${(1/2)*wheel_mass*radius*radius}"/>
+   value="${(1.0/12.0)*wheel_mass*(3*radius*radius + width*width)}"/>
 <xacro:property name="Iz_wheel"
-   value="${(1/12)*wheel_mass*(3*radius*radius + width*width)}"/>
+   value="${(0.5)*wheel_mass*radius*radius}"/>
 <!-- CASTOR LINK MOMENT OF INERTIA -->
 <xacro:property name = "Ix_castor"
-   value = "${(2/5)*castor_mass*radius*radius}" />
+   value = "${(2.0/5.0)*castor_mass*radius*radius}" />
 <xacro:property name = "Iy_castor"
-   value = "${(2/5)*castor_mass*radius*radius}" />
+   value = "${(2.0/5.0)*castor_mass*radius*radius}" />
 <xacro:property name = "Iz_castor"
-   value = "${(2/5)*castor_mass*radius*radius}" />
+   value = "${(2.0/5.0)*castor_mass*radius*radius}" />
 <!-- complete inertial system of the body -->
 <!-- FILE THAT INCLUDES GAZEBO OPTIONS AND MOTION CONTROLS-->

Commit message: minor change

File: src/mobile_robot/model/robot.xacro (robot description, xacro)
@@ -119,5 +119,5 @@
          <box size = "${body_length} ${body_height} ${body_width}"/>
       </geometry>
-      <origin r py = "0 0 0" xyz="0 0 ${s1}" />
+      <origin rpy = "0 0 0" xyz="0 0 ${s1}" />
    </collision>
    <xacro:body_link_macro/>

Commit message: minute errors resolved

File: src/mobile_robot/model/robot.xacro (robot description, xacro)
@@ -98,6 +98,4 @@
    </inertial>
 </xacro:macro>
-<!-- INERTFACE FOR COMTROLS -->
-<xacro:include filename="$(find mobile_robot)/model/robot.gazebo"/>
 <!-- FICTOUS LINK  -->
 <!-- DEFINING LINKS ANDS JOINTS -->
@@ -129,5 +127,5 @@
    <child link = "wheel1_link"/>
    <origin xyz= " ${-s2} ${-s4} ${radius}" rpy="0 0 0"/>
-   <axis xyz= "0 1 0"/>
+   <axis xyz= "0 0 1"/>
    <limit effort = "100000" velocity= "10"/>
    <dynamics damping ="1.0" friction ="1.0"/>
@@ -152,5 +150,5 @@
    <child link = "wheel2_link"/>
    <origin xyz= " ${-s2} ${s4} ${radius}" rpy="0 0 0"/>
-   <axis xyz= "0 1 0"/>
+   <axis xyz= "0 0 1"/>
    <limit effort = "100000" velocity= "10"/>
    <dynamics damping ="1.0" friction ="1.0"/>

Commit message: minute changes

File: src/mobile_robot/model/robot.xacro (robot description, xacro)
@@ -170,5 +170,5 @@
 </link>
 <!-- CASTOR JOINT -->
-<joint name="caster_joint" type ="continuous">
+<joint name="caster_joint" type ="fixed">
    <parent link = "body_link"/>
    <child link = "caster_link"/>

Commit message: minute error removal

File: src/mobile_robot/model/robot.xacro (robot description, xacro)
@@ -5,56 +5,35 @@
 <!-- BODY LINK DIMENSIONS  -->
 <!-- units used in meters -->
-<xacro:property name = "body_length"
-   value ="1.0"/>
-<xacro:property name = "body_width"
-   value ="0.3"/>
-<xacro:property name = "body_height"
-   value ="0.6"/>
+<xacro:property name = "body_length" value ="1.0"/>
+<xacro:property name = "body_width"  value ="0.6"/>
+<xacro:property name = "body_height" value ="0.3"/>
 <!-- WHEEL DIMENSIONS  AND CASTOR DIMENSIONS -->
-<!-- RADIUS -->
-<xacro:property name = "radius"
-   value = "0.15"/>
-<!-- WIDTH  WHEEL -->
-<xacro:property name ="width"
-   value ="0.1"/>
+<xacro:property name = "radius" value = "0.15"/>
+<xacro:property name ="width"  value ="0.1"/>
 <!-- other dimensions -->
-<xacro:property name = "s1"
-   value = "${body_width/2 + radius}"/>
-<xacro:property name = "s2"
-   value ="${radius*2}"/>
-<xacro:property name = "s3"
-   value = "${radius*2}"/>
-<xacro:property name = "s4"
-   value ="${body_height/2 + width/2}"/>
+<xacro:property name = "s1" value = "${body_height/2}"/>
+<!-- ✅ FIXED -->
+<xacro:property name = "s2" value ="${body_length/2 - radius}"/>
+<xacro:property name = "s3" value = "${radius*2}"/>
+<!-- ✅ FIXED -->
+<xacro:property name = "s4" value ="${body_width/2}"/>
 <!-- MASS NAD INERTIA -->
-<!-- DENSITY -->
-<!-- BODY LINK -->
-<xacro:property name = "body"
-   value = "2710.0"/>
-<!-- WHEEL LINK -->
-<xacro:property name = "wheel"
-   value = "2710.0"/>
-<!-- CASTOR LINK -->
-<xacro:property name = "castor"
-   value = "2710.0"/>
+<xacro:property name = "body"   value = "2710.0"/>
+<xacro:property name = "wheel"  value = "2710.0"/>
+<xacro:property name = "castor" value = "2710.0"/>
 <!-- MASS -->
-<!-- BODY LINK MASS -->
 <xacro:property name = "body_mass"
    value = "${body*body_length*body_width*body_height}"/>
-<!-- WHEEL LINK MASS -->
 <xacro:property name = "wheel_mass"
    value = "${wheel*ohm*radius*radius*width}"/>
-<!-- CASTOR LINK MASS -->
 <xacro:property name = "castor_mass"
    value = "${castor*(4.0/3.0)*ohm*radius*radius*radius}"/>
-<!--MOMENT OF INERTIA -->
-<!-- BODY LINK MOMENT OF INERTIA -->
+<!-- MOMENT OF INERTIA -->
 <xacro:property name = "Ix_body"
-   value = "${(1/12)*body_mass*(body_height*body_height + body_width*body_width)}" />
+   value = "${(1/12)*body_mass*(body_height*body_height + body_width*body_width)}"/>
 <xacro:property name = "Iy_body"
-   value = "${(1/12)*body_mass*(body_length*body_length + body_width*body_width)}" />
+   value = "${(1/12)*body_mass*(body_length*body_length + body_width*body_width)}"/>
 <xacro:property name = "Iz_body"
-   value = "${(1/12)*body_mass*(body_length*body_length + body_height*body_height)}" />
-<!-- WHEEL LINK MOMENT OF INERTIA -->
+   value = "${(1/12)*body_mass*(body_length*body_length + body_height*body_height)}"/>
 <xacro:property name="Ix_wheel"
    value="${(1.0/12.0)*wheel_mass*(3*radius*radius + width*width)}"/>
@@ -63,133 +42,96 @@
 <xacro:property name="Iz_wheel"
    value="${(0.5)*wheel_mass*radius*radius}"/>
-<!-- CASTOR LINK MOMENT OF INERTIA -->
 <xacro:property name = "Ix_castor"
-   value = "${(2.0/5.0)*castor_mass*radius*radius}" />
+   value = "${(2.0/5.0)*castor_mass*radius*radius}"/>
 <xacro:property name = "Iy_castor"
-   value = "${(2.0/5.0)*castor_mass*radius*radius}" />
+   value = "${(2.0/5.0)*castor_mass*radius*radius}"/>
 <xacro:property name = "Iz_castor"
-   value = "${(2.0/5.0)*castor_mass*radius*radius}" />
-<!-- complete inertial system of the body -->
-<!-- FILE THAT INCLUDES GAZEBO OPTIONS AND MOTION CONTROLS-->
+   value = "${(2.0/5.0)*castor_mass*radius*radius}"/>
 <xacro:include filename ="$(find mobile_robot)/model/robot.gazebo"/>
-<!-- THE BASIC COORDINATE SYSTEM IS CENTERED AT THE GEOMETRIC CENTER OF THE BODY LINK -->
-<!-- BODY LINK -->
-<xacro:macro name = "body_link_macro">
-   <inertial>
-   <origin rpy = "0 0 0" xyz = " 0 0 ${s1}"/>
-   <mass value = "${body_mass}"/>
-   <inertia ixx ="${Ix_body}" ixy = "0.0" ixz ="0.0" iyy ="${Iy_body}" iyz = "0.0" izz= "${Iz_body}"/>
-   </inertial>
-</xacro:macro>
-<!-- WHEEL LINK -->
-<xacro:macro name = "wheel_link_macro">
-   <inertial>
-   <origin rpy = " 1.570795 0 0" xyz = "0 0 0" />
-   <mass value = "${wheel_mass}"/>
-   <inertia ixx ="${Ix_wheel}" ixy="0.0" ixz="0.0" iyy="${Iy_wheel}" iyz ="0.0" izz="${Iz_wheel}"/>
-   </inertial>
-</xacro:macro>
-<!-- CASTOR LINK -->
-<xacro:macro name = "castor_link_macro">
-   <inertial>
-   <origin rpy = "0 0 0" xyz = "0 0 0" />
-   <mass value = "${castor_mass}"/>
-   <inertia ixx = "${Ix_castor}" ixy= "0.0" ixz="0.0" iyy="${Iy_castor}" iyz="0.0" izz= "${Iz_castor}"/>
-   </inertial>
-</xacro:macro>
-<!-- FICTOUS LINK  -->
-<!-- DEFINING LINKS ANDS JOINTS -->
-<link name  = "base_footprint"></link>
-<joint name = "body_link_joint" type = "fixed">
-   <parent link = "base_footprint"/>
-   <child link = "body_link"/>
-   <origin xyz= "0 0 0"/>
+<!-- BASE -->
+<link name="base_footprint"/>
+<joint name="body_link_joint" type="fixed">
+  <parent link="base_footprint"/>
+  <child link="body_link"/>
+  <origin xyz="0 0 0"/>
 </joint>
-<!-- BODY LINK OF ROBOT -->
-<link name = "body_link">
-   <visual>
-      <geometry>
-         <box size = "${body_length} ${body_height} ${body_width}"/>
-      </geometry>
-      <origin rpy = "0 0 0" xyz="0 0 ${s1}"/>
-   </visual>
-   <collision>
-      <geometry>
-         <box size = "${body_length} ${body_height} ${body_width}"/>
-      </geometry>
-      <origin rpy = "0 0 0" xyz="0 0 ${s1}" />
-   </collision>
-   <xacro:body_link_macro/>
+<!-- BODY -->
+<link name="body_link">
+  <visual>
+    <geometry>
+      <box size="${body_length} ${body_width} ${body_height}"/>
+    </geometry>
+    <origin xyz="0 0 ${s1}"/>
+  </visual>
+  <collision>
+    <geometry>
+      <box size="${body_length} ${body_width} ${body_height}"/>
+    </geometry>
+    <origin xyz="0 0 ${s1}"/>
+  </collision>
+  <xacro:body_link_macro/>
 </link>
-<!-- WHEEL JOINT -->
-<joint name="wheel1_joint" type ="continuous">
-   <parent link = "body_link"/>
-   <child link = "wheel1_link"/>
-   <origin xyz= " ${-s2} ${-s4} ${radius}" rpy="0 0 0"/>
-   <axis xyz= "0 0 1"/>
-   <limit effort = "100000" velocity= "10"/>
-   <dynamics damping ="1.0" friction ="1.0"/>
+<!-- LEFT WHEEL -->
+<joint name="wheel1_joint" type="continuous">
+  <parent link="body_link"/>
+  <child link="wheel1_link"/>
+  <origin xyz="${-s2} ${-s4} ${radius}"/>
+  <axis xyz="0 1 0"/>
 </joint>
-<link name = "wheel1_link">
-   <visual>
-      <geometry>
-         <cylinder length = "${width}" radius = "${radius}"/>
-      </geometry>
-      <origin xyz = "0 0 0" rpy = "1.570795 0 0"/>
-   </visual>
-   <collision>
-      <geometry>
-         <cylinder length = "${width}" radius = "${radius}"/>
-      </geometry>
-      <origin xyz = "0 0 0" rpy = "1.570795 0 0"/>
-   </collision>
-   <xacro:wheel_link_macro/>
+<link name="wheel1_link">
+  <visual>
+    <geometry>
+      <cylinder length="${width}" radius="${radius}"/>
+    </geometry>
+    <origin rpy="1.570795 0 0"/>
+  </visual>
+  <collision>
+    <geometry>
+      <cylinder length="${width}" radius="${radius}"/>
+    </geometry>
+    <origin rpy="1.570795 0 0"/>
+  </collision>
+  <xacro:wheel_link_macro/>
 </link>
-<joint name="wheel2_joint" type ="continuous">
-   <parent link = "body_link"/>
-   <child link = "wheel2_link"/>
-   <origin xyz= " ${-s2} ${s4} ${radius}" rpy="0 0 0"/>
-   <axis xyz= "0 0 1"/>
-   <limit effort = "100000" velocity= "10"/>
-   <dynamics damping ="1.0" friction ="1.0"/>
+<!-- RIGHT WHEEL -->
+<joint name="wheel2_joint" type="continuous">
+  <parent link="body_link"/>
+  <child link="wheel2_link"/>
+  <origin xyz="${-s2} ${s4} ${radius}"/>
+  <axis xyz="0 1 0"/>
 </joint>
-<link name = "wheel2_link">
-   <visual>
-      <geometry>
-         <cylinder length = "${width}" radius = "${radius}"/>
-      </geometry>
-      <origin xyz = "0 0 0" rpy = "1.570795 0 0"/>
-   </visual>
-   <collision>
-      <geometry>
-         <cylinder length = "${width}" radius = "${radius}"/>
-      </geometry>
-      <origin xyz = "0 0 0" rpy = "1.570795 0 0"/>
-   </collision>
-   <xacro:wheel_link_macro/>
+<link name="wheel2_link">
+  <visual>
+    <geometry>
+      <cylinder length="${width}" radius="${radius}"/>
+    </geometry>
+    <origin rpy="1.570795 0 0"/>
+  </visual>
+  <collision>
+    <geometry>
+      <cylinder length="${width}" radius="${radius}"/>
+    </geometry>
+    <origin rpy="1.570795 0 0"/>
+  </collision>
+  <xacro:wheel_link_macro/>
 </link>
-<!-- CASTOR JOINT -->
-<joint name="caster_joint" type ="continuous">
-   <parent link = "body_link"/>
-   <child link = "caster_link"/>
-   <origin xyz= " ${body_length/2 - radius} 0 ${radius}" rpy="0 0 0"/>
-   <axis xyz= "0 1 0"/>
-   <limit effort = "100000" velocity= "10"/>
-   <dynamics damping ="1.0" friction ="1.0"/>
+<!-- CASTER -->
+<joint name="caster_joint" type="fixed">
+  <parent link="body_link"/>
+  <child link="caster_link"/>
+  <origin xyz="${body_length/2 - radius} 0 ${radius}"/>
 </joint>
-<link name = "caster_link">
-   <visual>
-      <geometry>
-         <sphere radius = "${radius}"/>
-      </geometry>
-      <origin xyz = "0 0 0" rpy = "0 0 0"/>
-   </visual>
-   <collision>
-      <geometry>
-         <sphere radius = "${radius}"/>
-      </geometry>
-      <origin xyz = "0 0 0" rpy = "0 0 0"/>
-   </collision>
-   <xacro:castor_link_macro/>
+<link name="caster_link">
+  <visual>
+    <geometry>
+      <sphere radius="${radius}"/>
+    </geometry>
+  </visual>
+  <collision>
+    <geometry>
+      <sphere radius="${radius}"/>
+    </geometry>
+  </collision>
+  <xacro:castor_link_macro/>
 </link>
 </robot>

Commit message: changes reolsved

File: src/mobile_robot/model/robot.xacro (robot description, xacro)
@@ -49,4 +49,36 @@
    value = "${(2.0/5.0)*castor_mass*radius*radius}"/>
 <xacro:include filename ="$(find mobile_robot)/model/robot.gazebo"/>
+<!-- ================= INERTIAL MACROS ================= -->
+<!-- BODY LINK -->
+<xacro:macro name="body_link_macro">
+  <inertial>
+    <origin xyz="0 0 ${s1}"/>
+    <mass value="${body_mass}"/>
+    <inertia
+      ixx="${Ix_body}" ixy="0" ixz="0"
+      iyy="${Iy_body}" iyz="0"
+      izz="${Iz_body}"/>
+  </inertial>
+</xacro:macro>
+<!-- WHEEL LINK -->
+<xacro:macro name="wheel_link_macro">
+  <inertial>
+    <mass value="${wheel_mass}"/>
+    <inertia
+      ixx="${Ix_wheel}" ixy="0" ixz="0"
+      iyy="${Iy_wheel}" iyz="0"
+      izz="${Iz_wheel}"/>
+  </inertial>
+</xacro:macro>
+<!-- CASTER LINK -->
+<xacro:macro name="castor_link_macro">
+  <inertial>
+    <mass value="${castor_mass}"/>
+    <inertia
+      ixx="${Ix_castor}" ixy="0" ixz="0"
+      iyy="${Iy_castor}" iyz="0"
+      izz="${Iz_castor}"/>
+  </inertial>
+</xacro:macro>
 <!-- BASE -->
 <link name="base_footprint"/>

Commit message: latest run to see the errors

File: src/mobile_robot/model/robot.xacro (robot description, xacro)
@@ -152,5 +152,5 @@
   <parent link="body_link"/>
   <child link="caster_link"/>
-  <origin xyz="${body_length/2 - radius} 0 ${radius}"/>
+  <origin xyz="${s1} 0 ${radius}"/>
 </joint>
 <link name="caster_link">
