Commit message: latest run

File: src/mobile_robot/model/robot.xacro (robot description, xacro)
@@ -1,57 +1,56 @@
-<?xml version='1.0'?>
-<robot name = "castor_robot" xmlns:xacro="http://www.ros.org/wiki/xacro">
-<!-- define constants -->
-<xacro:property name = "ohm" value ="3.14159"/>
-<!-- BODY LINK DIMENSIONS  -->
-<!-- units used in meters -->
-<xacro:property name = "body_length" value ="1.0"/>
-<xacro:property name = "body_width"  value ="0.6"/>
-<xacro:property name = "body_height" value ="0.3"/>
-<!-- WHEEL DIMENSIONS  AND CASTOR DIMENSIONS -->
-<xacro:property name = "radius" value = "0.15"/>
-<xacro:property name ="width"  value ="0.1"/>
-<!-- other dimensions -->
-<xacro:property name = "s1" value = "${body_height/2}"/>
-<!-- ✅ FIXED -->
-<xacro:property name = "s2" value ="${body_length/2 - radius}"/>
-<xacro:property name = "s3" value = "${radius*2}"/>
-<!-- ✅ FIXED -->
-<xacro:property name = "s4" value ="${body_width/2}"/>
-<!-- MASS NAD INERTIA -->
-<xacro:property name = "body"   value = "2710.0"/>
-<xacro:property name = "wheel"  value = "2710.0"/>
-<xacro:property name = "castor" value = "2710.0"/>
-<!-- MASS -->
-<xacro:property name = "body_mass"
-   value = "${body*body_length*body_width*body_height}"/>
-<xacro:property name = "wheel_mass"
-   value = "${wheel*ohm*radius*radius*width}"/>
-<xacro:property name = "castor_mass"
-   value = "${castor*(4.0/3.0)*ohm*radius*radius*radius}"/>
-<!-- MOMENT OF INERTIA -->
-<xacro:property name = "Ix_body"
-   value = "${(1/12)*body_mass*(body_height*body_height + body_width*body_width)}"/>
-<xacro:property name = "Iy_body"
-   value = "${(1/12)*body_mass*(body_length*body_length + body_width*body_width)}"/>
-<xacro:property name = "Iz_body"
-   value = "${(1/12)*body_mass*(body_length*body_length + body_height*body_height)}"/>
+<?xml version="1.0"?>
+<robot name="castor_robot" xmlns:xacro="http://www.ros.org/wiki/xacro">
+<!-- ========================================================= -->
+<!-- ===================== CONSTANTS ========================= -->
+<!-- ========================================================= -->
+<xacro:property name="pi" value="3.141592653589793"/>
+<!-- ================= BODY DIMENSIONS (meters) =============== -->
+<xacro:property name="body_length" value="1.0"/>
+<xacro:property name="body_width"  value="0.6"/>
+<xacro:property name="body_height" value="0.3"/>
+<!-- ================= WHEEL DIMENSIONS ======================= -->
+<xacro:property name="radius" value="0.15"/>
+<xacro:property name="width"  value="0.1"/>
+<!-- ================= GEOMETRIC OFFSETS (MATCH DIAGRAM) ====== -->
+<!-- vertical -->
+<xacro:property name="z_wheel" value="${radius}"/>
+<xacro:property name="z_body"  value="${radius + body_height/2}"/>
+<!-- longitudinal -->
+<xacro:property name="x_wheel"  value="${-body_length/2 + radius}"/>
+<xacro:property name="x_caster" value="${ body_length/2 - radius}"/>
+<!-- lateral -->
+<xacro:property name="y_wheel" value="${body_width/2 + width/2}"/>
+<!-- ========================================================= -->
+<!-- ======================= MASS ============================ -->
+<!-- ========================================================= -->
+<xacro:property name="body_mass"   value="25.0"/>
+<xacro:property name="wheel_mass"  value="1.5"/>
+<xacro:property name="caster_mass" value="0.5"/>
+<!-- ========================================================= -->
+<!-- ===================== INERTIA ============================ -->
+<!-- ========================================================= -->
+<!-- BODY -->
+<xacro:property name="Ix_body"
+  value="${(1/12)*body_mass*(body_height*body_height + body_width*body_width)}"/>
+<xacro:property name="Iy_body"
+  value="${(1/12)*body_mass*(body_length*body_length + body_width*body_width)}"/>
+<xacro:property name="Iz_body"
+  value="${(1/12)*body_mass*(body_length*body_length + body_height*body_height)}"/>
+<!-- WHEEL -->
 <xacro:property name="Ix_wheel"
-   value="${(1.0/12.0)*wheel_mass*(3*radius*radius + width*width)}"/>
+  value="${(1/12)*wheel_mass*(3*radius*radius + width*width)}"/>
 <xacro:property name="Iy_wheel"
-   value="${(1.0/12.0)*wheel_mass*(3*radius*radius + width*width)}"/>
+  value="${(1/12)*wheel_mass*(3*radius*radius + width*width)}"/>
 <xacro:property name="Iz_wheel"
-   value="${(0.5)*wheel_mass*radius*radius}"/>
-<xacro:property name = "Ix_castor"
-   value = "${(2.0/5.0)*castor_mass*radius*radius}"/>
-<xacro:property name = "Iy_castor"
-   value = "${(2.0/5.0)*castor_mass*radius*radius}"/>
-<xacro:property name = "Iz_castor"
-   value = "${(2.0/5.0)*castor_mass*radius*radius}"/>
-<xacro:include filename ="$(find mobile_robot)/model/robot.gazebo"/>
-<!-- ================= INERTIAL MACROS ================= -->
-<!-- BODY LINK -->
-<xacro:macro name="body_link_macro">
+  value="${0.5*wheel_mass*radius*radius}"/>
+<!-- CASTER -->
+<xacro:property name="I_caster"
+  value="${(2/5)*caster_mass*radius*radius}"/>
+<!-- ========================================================= -->
+<!-- ==================== INERTIAL MACROS ==================== -->
+<!-- ========================================================= -->
+<xacro:macro name="body_inertial">
   <inertial>
-    <origin xyz="0 0 ${s1}"/>
+    <origin xyz="0 0 ${z_body}"/>
     <mass value="${body_mass}"/>
     <inertia
@@ -61,6 +60,5 @@
   </inertial>
 </xacro:macro>
-<!-- WHEEL LINK -->
-<xacro:macro name="wheel_link_macro">
+<xacro:macro name="wheel_inertial">
   <inertial>
     <mass value="${wheel_mass}"/>
@@ -71,22 +69,25 @@
   </inertial>
 </xacro:macro>
-<!-- CASTER LINK -->
-<xacro:macro name="castor_link_macro">
+<xacro:macro name="caster_inertial">
   <inertial>
-    <mass value="${castor_mass}"/>
+    <mass value="${caster_mass}"/>
     <inertia
-      ixx="${Ix_castor}" ixy="0" ixz="0"
-      iyy="${Iy_castor}" iyz="0"
-      izz="${Iz_castor}"/>
+      ixx="${I_caster}" ixy="0" ixz="0"
+      iyy="${I_caster}" iyz="0"
+      izz="${I_caster}"/>
   </inertial>
 </xacro:macro>
-<!-- BASE -->
+<!-- ========================================================= -->
+<!-- ====================== BASE ============================== -->
+<!-- ========================================================= -->
 <link name="base_footprint"/>
-<joint name="body_link_joint" type="fixed">
+<joint name="base_to_body" type="fixed">
   <parent link="base_footprint"/>
   <child link="body_link"/>
   <origin xyz="0 0 0"/>
 </joint>
-<!-- BODY -->
+<!-- ========================================================= -->
+<!-- ====================== BODY ============================== -->
+<!-- ========================================================= -->
 <link name="body_link">
   <visual>
@@ -94,5 +95,5 @@
       <box size="${body_length} ${body_width} ${body_height}"/>
     </geometry>
-    <origin xyz="0 0 ${s1}"/>
+    <origin xyz="0 0 ${z_body}"/>
   </visual>
   <collision>
@@ -100,70 +101,78 @@
       <box size="${body_length} ${body_width} ${body_height}"/>
     </geometry>
-    <origin xyz="0 0 ${s1}"/>
+    <origin xyz="0 0 ${z_body}"/>
   </collision>
-  <xacro:body_link_macro/>
+  <xacro:body_inertial/>
 </link>
-<!-- LEFT WHEEL -->
-<joint name="wheel1_joint" type="continuous">
+<!-- ========================================================= -->
+<!-- ====================== LEFT WHEEL ======================= -->
+<!-- ========================================================= -->
+<joint name="wheel_left_joint" type="continuous">
   <parent link="body_link"/>
-  <child link="wheel1_link"/>
-  <origin xyz="${-s2} ${-s4} ${radius}"/>
+  <child link="wheel_left_link"/>
+  <origin xyz="${x_wheel} ${ y_wheel} ${z_wheel}"/>
   <axis xyz="0 1 0"/>
 </joint>
-<link name="wheel1_link">
+<link name="wheel_left_link">
   <visual>
     <geometry>
-      <cylinder length="${width}" radius="${radius}"/>
+      <cylinder radius="${radius}" length="${width}"/>
     </geometry>
-    <origin rpy="1.570795 0 0"/>
+    <origin rpy="1.5708 0 0"/>
   </visual>
   <collision>
     <geometry>
-      <cylinder length="${width}" radius="${radius}"/>
+      <cylinder radius="${radius}" length="${width}"/>
     </geometry>
-    <origin rpy="1.570795 0 0"/>
+    <origin rpy="1.5708 0 0"/>
   </collision>
-  <xacro:wheel_link_macro/>
+  <xacro:wheel_inertial/>
 </link>
-<!-- RIGHT WHEEL -->
-<joint name="wheel2_joint" type="continuous">
+<!-- ========================================================= -->
+<!-- ====================== RIGHT WHEEL ====================== -->
+<!-- ========================================================= -->
+<joint name="wheel_right_joint" type="continuous">
   <parent link="body_link"/>
-  <child link="wheel2_link"/>
-  <origin xyz="${-s2} ${s4} ${radius}"/>
+  <child link="wheel_right_link"/>
+  <origin xyz="${x_wheel} ${-y_wheel} ${z_wheel}"/>
   <axis xyz="0 1 0"/>
 </joint>
-<link name="wheel2_link">
+<link name="wheel_right_link">
   <visual>
     <geometry>
-      <cylinder length="${width}" radius="${radius}"/>
+      <cylinder radius="${radius}" length="${width}"/>
     </geometry>
-    <origin rpy="1.570795 0 0"/>
+    <origin rpy="1.5708 0 0"/>
   </visual>
   <collision>
     <geometry>
-      <cylinder length="${width}" radius="${radius}"/>
+      <cylinder radius="${radius}" length="${width}"/>
     </geometry>
-    <origin rpy="1.570795 0 0"/>
+    <origin rpy="1.5708 0 0"/>
   </collision>
-  <xacro:wheel_link_macro/>
+  <xacro:wheel_inertial/>
 </link>
-<!-- CASTER -->
+<!-- ========================================================= -->
+<!-- ====================== CASTER =========================== -->
+<!-- ========================================================= -->
 <joint name="caster_joint" type="fixed">
   <parent link="body_link"/>
   <child link="caster_link"/>
-  <origin xyz="${s1} 0 ${radius}"/>
+  <origin xyz="${x_caster} 0 ${z_wheel}"/>
 </joint>
 <link name="caster_link">
   <visual>
     <geometry>
-      <sphere radius="${radius}"/>
+      <cylinder radius="0.05" length="0.02"/>
     </geometry>
+    <origin rpy="1.5708 0 0"/>
   </visual>
   <collision>
     <geometry>
-      <sphere radius="${radius}"/>
+      <cylinder radius="0.05" length="0.02"/>
     </geometry>
+    <origin rpy="1.5708 0 0"/>
   </collision>
-  <xacro:castor_link_macro/>
+  <xacro:caster_inertial/>
 </link>
 </robot>

Commit message: sorting the issues

File: src/mobile_robot/model/robot.xacro (robot description, xacro)
@@ -12,11 +12,14 @@
 <xacro:property name="radius" value="0.15"/>
 <xacro:property name="width"  value="0.1"/>
-<!-- ================= GEOMETRIC OFFSETS (MATCH DIAGRAM) ====== -->
+<!-- ========================================================= -->
+<!-- ========== GEOMETRIC OFFSETS (MATCH DIAGRAM) ============= -->
+<!-- ========================================================= -->
 <!-- vertical -->
 <xacro:property name="z_wheel" value="${radius}"/>
 <xacro:property name="z_body"  value="${radius + body_height/2}"/>
 <!-- longitudinal -->
+<!-- caster is at FRONT (+X), wheels are behind -->
+<xacro:property name="x_caster" value="${ body_length/2 - radius}"/>
 <xacro:property name="x_wheel"  value="${-body_length/2 + radius}"/>
-<xacro:property name="x_caster" value="${ body_length/2 - radius}"/>
 <!-- lateral -->
 <xacro:property name="y_wheel" value="${body_width/2 + width/2}"/>
@@ -154,5 +157,5 @@
 </link>
 <!-- ========================================================= -->
-<!-- ====================== CASTER =========================== -->
+<!-- ====================== FRONT CASTER ==================== -->
 <!-- ========================================================= -->
 <joint name="caster_joint" type="fixed">
@@ -164,5 +167,7 @@
   <visual>
     <geometry>
-      <cylinder radius="0.05" length="0.02"/>
+      <geometry>
+        <sphere radius="${radius}"/>
+      </geometry>
     </geometry>
     <origin rpy="1.5708 0 0"/>
@@ -170,5 +175,5 @@
   <collision>
     <geometry>
-      <cylinder radius="0.05" length="0.02"/>
+        <sphere radius="${radius}"/>
     </geometry>
     <origin rpy="1.5708 0 0"/>
