Commit message: corrected xacro

File: src/mobile_robot/model/robot.xacro (robot description, xacro)
@@ -1,183 +1,195 @@
-<?xml version="1.0"?>
-<robot name="castor_robot" xmlns:xacro="http://www.ros.org/wiki/xacro">
-<!-- ========================================================= -->
-<!-- ===================== CONSTANTS ========================= -->
-<!-- ========================================================= -->
-<xacro:property name="pi" value="3.141592653589793"/>
-<!-- ================= BODY DIMENSIONS (meters) =============== -->
-<xacro:property name="body_length" value="1.0"/>
-<xacro:property name="body_width"  value="0.6"/>
-<xacro:property name="body_height" value="0.3"/>
-<!-- ================= WHEEL DIMENSIONS ======================= -->
-<xacro:property name="radius" value="0.15"/>
-<xacro:property name="width"  value="0.1"/>
-<!-- ========================================================= -->
-<!-- ========== GEOMETRIC OFFSETS (MATCH DIAGRAM) ============= -->
-<!-- ========================================================= -->
-<!-- vertical -->
-<xacro:property name="z_wheel" value="${radius}"/>
-<xacro:property name="z_body"  value="${radius + body_height/2}"/>
-<!-- longitudinal -->
-<!-- caster is at FRONT (+X), wheels are behind -->
-<xacro:property name="x_caster" value="${ body_length/2 - radius}"/>
-<xacro:property name="x_wheel"  value="${-body_length/2 + radius}"/>
-<!-- lateral -->
-<xacro:property name="y_wheel" value="${body_width/2 + width/2}"/>
-<!-- ========================================================= -->
-<!-- ======================= MASS ============================ -->
-<!-- ========================================================= -->
-<xacro:property name="body_mass"   value="25.0"/>
-<xacro:property name="wheel_mass"  value="1.5"/>
-<xacro:property name="caster_mass" value="0.5"/>
-<!-- ========================================================= -->
-<!-- ===================== INERTIA ============================ -->
-<!-- ========================================================= -->
-<!-- BODY -->
-<xacro:property name="Ix_body"
-  value="${(1/12)*body_mass*(body_height*body_height + body_width*body_width)}"/>
-<xacro:property name="Iy_body"
-  value="${(1/12)*body_mass*(body_length*body_length + body_width*body_width)}"/>
-<xacro:property name="Iz_body"
-  value="${(1/12)*body_mass*(body_length*body_length + body_height*body_height)}"/>
-<!-- WHEEL -->
+<?xml version='1.0'?>
+<robot name = "castor_robot" xmlns:xacro="http://www.ros.org/wiki/xacro">
+<!-- define constants -->
+<xacro:property name = "ohm" value ="3.14159"/>
+<!-- BODY LINK DIMENSIONS  -->
+<!-- units used in meters -->
+<xacro:property name = "body_length"
+   value ="1.0"/>
+<xacro:property name = "body_width"
+   value ="0.3"/>
+<xacro:property name = "body_height"
+   value ="0.6"/>
+<!-- WHEEL DIMENSIONS  AND CASTOR DIMENSIONS -->
+<!-- RADIUS -->
+<xacro:property name = "radius"
+   value = "0.15"/>
+<!-- WIDTH  WHEEL -->
+<xacro:property name ="width"
+   value ="0.1"/>
+<!-- other dimensions -->
+<xacro:property name = "s1"
+   value = "${body_width/2 + radius}"/>
+<xacro:property name = "s2"
+   value ="${radius*2}"/>
+<xacro:property name = "s3"
+   value = "${radius*2}"/>
+<xacro:property name = "s4"
+   value ="${body_height/2 + width/2}"/>
+<!-- MASS NAD INERTIA -->
+<!-- DENSITY -->
+<!-- BODY LINK -->
+<xacro:property name = "body"
+   value = "2710.0"/>
+<!-- WHEEL LINK -->
+<xacro:property name = "wheel"
+   value = "2710.0"/>
+<!-- CASTOR LINK -->
+<xacro:property name = "castor"
+   value = "2710.0"/>
+<!-- MASS -->
+<!-- BODY LINK MASS -->
+<xacro:property name = "body_mass"
+   value = "${body*body_length*body_width*body_height}"/>
+<!-- WHEEL LINK MASS -->
+<xacro:property name = "wheel_mass"
+   value = "${wheel*ohm*radius*radius*width}"/>
+<!-- CASTOR LINK MASS -->
+<xacro:property name = "castor_mass"
+   value = "${castor*(4.0/3.0)*ohm*radius*radius*radius}"/>
+<!--MOMENT OF INERTIA -->
+<!-- BODY LINK MOMENT OF INERTIA -->
+<xacro:property name = "Ix_body"
+   value = "${(1/12)*body_mass*(body_height*body_height + body_width*body_width)}" />
+<xacro:property name = "Iy_body"
+   value = "${(1/12)*body_mass*(body_length*body_length + body_width*body_width)}" />
+<xacro:property name = "Iz_body"
+   value = "${(1/12)*body_mass*(body_length*body_length + body_height*body_height)}" />
+<!-- WHEEL LINK MOMENT OF INERTIA -->
 <xacro:property name="Ix_wheel"
-  value="${(1/12)*wheel_mass*(3*radius*radius + width*width)}"/>
+   value="${(1.0/12.0)*wheel_mass*(3*radius*radius + width*width)}"/>
 <xacro:property name="Iy_wheel"
-  value="${(1/12)*wheel_mass*(3*radius*radius + width*width)}"/>
+   value="${(1.0/12.0)*wheel_mass*(3*radius*radius + width*width)}"/>
 <xacro:property name="Iz_wheel"
-  value="${0.5*wheel_mass*radius*radius}"/>
-<!-- CASTER -->
-<xacro:property name="I_caster"
-  value="${(2/5)*caster_mass*radius*radius}"/>
-<!-- ========================================================= -->
-<!-- ==================== INERTIAL MACROS ==================== -->
-<!-- ========================================================= -->
-<xacro:macro name="body_inertial">
-  <inertial>
-    <origin xyz="0 0 ${z_body}"/>
-    <mass value="${body_mass}"/>
-    <inertia
-      ixx="${Ix_body}" ixy="0" ixz="0"
-      iyy="${Iy_body}" iyz="0"
-      izz="${Iz_body}"/>
-  </inertial>
+   value="${(0.5)*wheel_mass*radius*radius}"/>
+<!-- CASTOR LINK MOMENT OF INERTIA -->
+<xacro:property name = "Ix_castor"
+   value = "${(2.0/5.0)*castor_mass*radius*radius}" />
+<xacro:property name = "Iy_castor"
+   value = "${(2.0/5.0)*castor_mass*radius*radius}" />
+<xacro:property name = "Iz_castor"
+   value = "${(2.0/5.0)*castor_mass*radius*radius}" />
+<!-- complete inertial system of the body -->
+<!-- FILE THAT INCLUDES GAZEBO OPTIONS AND MOTION CONTROLS-->
+<xacro:include filename ="$(find mobile_robot)/model/robot.gazebo"/>
+<!-- THE BASIC COORDINATE SYSTEM IS CENTERED AT THE GEOMETRIC CENTER OF THE BODY LINK -->
+<!-- BODY LINK -->
+<xacro:macro name = "body_link_macro">
+   <inertial>
+   <origin rpy = "0 0 0" xyz = " 0 0 ${s1}"/>
+   <mass value = "${body_mass}"/>
+   <inertia ixx ="${Ix_body}" ixy = "0.0" ixz ="0.0" iyy ="${Iy_body}" iyz = "0.0" izz= "${Iz_body}"/>
+   </inertial>
 </xacro:macro>
-<xacro:macro name="wheel_inertial">
-  <inertial>
-    <mass value="${wheel_mass}"/>
-    <inertia
-      ixx="${Ix_wheel}" ixy="0" ixz="0"
-      iyy="${Iy_wheel}" iyz="0"
-      izz="${Iz_wheel}"/>
-  </inertial>
+<!-- WHEEL LINK -->
+<xacro:macro name = "wheel_link_macro">
+   <inertial>
+   <origin rpy = " 1.570795 0 0" xyz = "0 0 0" />
+   <mass value = "${wheel_mass}"/>
+   <inertia ixx ="${Ix_wheel}" ixy="0.0" ixz="0.0" iyy="${Iy_wheel}" iyz ="0.0" izz="${Iz_wheel}"/>
+   </inertial>
 </xacro:macro>
-<xacro:macro name="caster_inertial">
-  <inertial>
-    <mass value="${caster_mass}"/>
-    <inertia
-      ixx="${I_caster}" ixy="0" ixz="0"
-      iyy="${I_caster}" iyz="0"
-      izz="${I_caster}"/>
-  </inertial>
+<!-- CASTOR LINK -->
+<xacro:macro name = "castor_link_macro">
+   <inertial>
+   <origin rpy = "0 0 0" xyz = "0 0 0" />
+   <mass value = "${castor_mass}"/>
+   <inertia ixx = "${Ix_castor}" ixy= "0.0" ixz="0.0" iyy="${Iy_castor}" iyz="0.0" izz= "${Iz_castor}"/>
+   </inertial>
 </xacro:macro>
-<!-- ========================================================= -->
-<!-- ====================== BASE ============================== -->
-<!-- ========================================================= -->
-<link name="base_footprint"/>
-<joint name="base_to_body" type="fixed">
-  <parent link="base_footprint"/>
-  <child link="body_link"/>
-  <origin xyz="0 0 0"/>
+<!-- FICTOUS LINK  -->
+<!-- DEFINING LINKS ANDS JOINTS -->
+<link name  = "base_footprint"></link>
+<joint name = "body_link_joint" type = "fixed">
+   <parent link = "base_footprint"/>
+   <child link = "body_link"/>
+   <origin xyz= "0 0 0"/>
 </joint>
-<!-- ========================================================= -->
-<!-- ====================== BODY ============================== -->
-<!-- ========================================================= -->
-<link name="body_link">
-  <visual>
-    <geometry>
-      <box size="${body_length} ${body_width} ${body_height}"/>
-    </geometry>
-    <origin xyz="0 0 ${z_body}"/>
-  </visual>
-  <collision>
-    <geometry>
-      <box size="${body_length} ${body_width} ${body_height}"/>
-    </geometry>
-    <origin xyz="0 0 ${z_body}"/>
-  </collision>
-  <xacro:body_inertial/>
+<!-- BODY LINK OF ROBOT -->
+<link name = "body_link">
+   <visual>
+      <geometry>
+         <box size = "${body_length} ${body_height} ${body_width}"/>
+      </geometry>
+      <origin rpy = "0 0 0" xyz="0 0 ${s1}"/>
+   </visual>
+   <collision>
+      <geometry>
+         <box size = "${body_length} ${body_height} ${body_width}"/>
+      </geometry>
+      <origin rpy = "0 0 0" xyz="0 0 ${s1}" />
+   </collision>
+   <xacro:body_link_macro/>
 </link>
-<!-- ========================================================= -->
-<!-- ====================== LEFT WHEEL ======================= -->
-<!-- ========================================================= -->
-<joint name="wheel_left_joint" type="continuous">
-  <parent link="body_link"/>
-  <child link="wheel_left_link"/>
-  <origin xyz="${x_wheel} ${ y_wheel} ${z_wheel}"/>
-  <axis xyz="0 1 0"/>
+<!-- WHEEL JOINT -->
+<joint name="wheel1_joint" type ="continuous">
+   <parent link = "body_link"/>
+   <child link = "wheel1_link"/>
+   <origin xyz= " ${-s2} ${-s4} ${radius}" rpy="0 0 0"/>
+   <axis xyz= "0 0 1"/>
+   <limit effort = "100000" velocity= "10"/>
+   <dynamics damping ="1.0" friction ="1.0"/>
 </joint>
-<link name="wheel_left_link">
-  <visual>
-    <geometry>
-      <cylinder radius="${radius}" length="${width}"/>
-    </geometry>
-    <origin rpy="1.5708 0 0"/>
-  </visual>
-  <collision>
-    <geometry>
-      <cylinder radius="${radius}" length="${width}"/>
-    </geometry>
-    <origin rpy="1.5708 0 0"/>
-  </collision>
-  <xacro:wheel_inertial/>
+<link name = "wheel1_link">
+   <visual>
+      <geometry>
+         <cylinder length = "${width}" radius = "${radius}"/>
+      </geometry>
+      <origin xyz = "0 0 0" rpy = "1.570795 0 0"/>
+   </visual>
+   <collision>
+      <geometry>
+         <cylinder length = "${width}" radius = "${radius}"/>
+      </geometry>
+      <origin xyz = "0 0 0" rpy = "1.570795 0 0"/>
+   </collision>
+   <xacro:wheel_link_macro/>
 </link>
-<!-- ========================================================= -->
-<!-- ====================== RIGHT WHEEL ====================== -->
-<!-- ========================================================= -->
-<joint name="wheel_right_joint" type="continuous">
-  <parent link="body_link"/>
-  <child link="wheel_right_link"/>
-  <origin xyz="${x_wheel} ${-y_wheel} ${z_wheel}"/>
-  <axis xyz="0 1 0"/>
+<joint name="wheel2_joint" type ="continuous">
+   <parent link = "body_link"/>
+   <child link = "wheel2_link"/>
+   <origin xyz= " ${-s2} ${s4} ${radius}" rpy="0 0 0"/>
+   <axis xyz= "0 0 1"/>
+   <limit effort = "100000" velocity= "10"/>
+   <dynamics damping ="1.0" friction ="1.0"/>
 </joint>
-<link name="wheel_right_link">
-  <visual>
-    <geometry>
-      <cylinder radius="${radius}" length="${width}"/>
-    </geometry>
-    <origin rpy="1.5708 0 0"/>
-  </visual>
-  <collision>
-    <geometry>
-      <cylinder radius="${radius}" length="${width}"/>
-    </geometry>
-    <origin rpy="1.5708 0 0"/>
-  </collision>
-  <xacro:wheel_inertial/>
+<link name = "wheel2_link">
+   <visual>
+      <geometry>
+         <cylinder length = "${width}" radius = "${radius}"/>
+      </geometry>
+      <origin xyz = "0 0 0" rpy = "1.570795 0 0"/>
+   </visual>
+   <collision>
+      <geometry>
+         <cylinder length = "${width}" radius = "${radius}"/>
+      </geometry>
+      <origin xyz = "0 0 0" rpy = "1.570795 0 0"/>
+   </collision>
+   <xacro:wheel_link_macro/>
 </link>
-<!-- ========================================================= -->
-<!-- ====================== FRONT CASTER ==================== -->
-<!-- ========================================================= -->
-<joint name="caster_joint" type="fixed">
-  <parent link="body_link"/>
-  <child link="caster_link"/>
-  <origin xyz="${x_caster} 0 ${z_wheel}"/>
+<!-- CASTOR JOINT -->
+<joint name="caster_joint" type ="continuous">
+   <parent link = "body_link"/>
+   <child link = "caster_link"/>
+   <origin xyz= " ${body_length/2 - radius} 0 ${radius}" rpy="0 0 0"/>
+   <axis xyz= "0 1 0"/>
+   <limit effort = "100000" velocity= "10"/>
+   <dynamics damping ="1.0" friction ="1.0"/>
 </joint>
-<link name="caster_link">
-  <visual>
-    <geometry>
+<link name = "caster_link">
+   <visual>
       <geometry>
-        <sphere radius="${radius}"/>
+         <sphere radius = "${radius}"/>
       </geometry>
-    </geometry>
-    <origin rpy="1.5708 0 0"/>
-  </visual>
-  <collision>
-    <geometry>
-        <sphere radius="${radius}"/>
-    </geometry>
-    <origin rpy="1.5708 0 0"/>
-  </collision>
-  <xacro:caster_inertial/>
+      <origin xyz = "0 0 0" rpy = "0 0 0"/>
+   </visual>
+   <collision>
+      <geometry>
+         <sphere radius = "${radius}"/>
+      </geometry>
+      <origin xyz = "0 0 0" rpy = "0 0 0"/>
+   </collision>
+   <xacro:castor_link_macro/>
 </link>
 </robot>

Commit message: latest run

File: src/mobile_robot/model/robot.xacro (robot description, xacro)
@@ -20,5 +20,5 @@
 <!-- other dimensions -->
 <xacro:property name = "s1"
-   value = "${body_width/2 + radius}"/>
+   value = "${body_height/2 + radius}"/>
 <xacro:property name = "s2"
    value ="${radius*2}"/>
@@ -26,26 +26,26 @@
    value = "${radius*2}"/>
 <xacro:property name = "s4"
-   value ="${body_height/2 + width/2}"/>
+   value ="${body_width/2 + width/2}"/>
 <!-- MASS NAD INERTIA -->
 <!-- DENSITY -->
 <!-- BODY LINK -->
-<xacro:property name = "body"
+<xacro:property name = "body_link"
    value = "2710.0"/>
 <!-- WHEEL LINK -->
-<xacro:property name = "wheel"
+<xacro:property name = "wheel_link"
    value = "2710.0"/>
 <!-- CASTOR LINK -->
-<xacro:property name = "castor"
+<xacro:property name = "castor_link"
    value = "2710.0"/>
 <!-- MASS -->
 <!-- BODY LINK MASS -->
 <xacro:property name = "body_mass"
-   value = "${body*body_length*body_width*body_height}"/>
+   value = "${body_link*body_length*body_width*body_height}"/>
 <!-- WHEEL LINK MASS -->
 <xacro:property name = "wheel_mass"
-   value = "${wheel*ohm*radius*radius*width}"/>
+   value = "${wheel_link*ohm*radius*radius*width}"/>
 <!-- CASTOR LINK MASS -->
 <xacro:property name = "castor_mass"
-   value = "${castor*(4.0/3.0)*ohm*radius*radius*radius}"/>
+   value = "${castor_link*(4/3)*ohm*radius*radius*radius}"/>
 <!--MOMENT OF INERTIA -->
 <!-- BODY LINK MOMENT OF INERTIA -->
@@ -58,16 +58,16 @@
 <!-- WHEEL LINK MOMENT OF INERTIA -->
 <xacro:property name="Ix_wheel"
-   value="${(1.0/12.0)*wheel_mass*(3*radius*radius + width*width)}"/>
+   value="${(1/12)*wheel_mass*(3*radius*radius + width*width)}"/>
 <xacro:property name="Iy_wheel"
-   value="${(1.0/12.0)*wheel_mass*(3*radius*radius + width*width)}"/>
+   value="${(1/2)*wheel_mass*radius*radius}"/>
 <xacro:property name="Iz_wheel"
-   value="${(0.5)*wheel_mass*radius*radius}"/>
+   value="${(1/12)*wheel_mass*(3*radius*radius + width*width)}"/>
 <!-- CASTOR LINK MOMENT OF INERTIA -->
 <xacro:property name = "Ix_castor"
-   value = "${(2.0/5.0)*castor_mass*radius*radius}" />
+   value = "${(2/5)*castor_mass*radius*radius}" />
 <xacro:property name = "Iy_castor"
-   value = "${(2.0/5.0)*castor_mass*radius*radius}" />
+   value = "${(2/5)*castor_mass*radius*radius}" />
 <xacro:property name = "Iz_castor"
-   value = "${(2.0/5.0)*castor_mass*radius*radius}" />
+   value = "${(2/5)*castor_mass*radius*radius}" />
 <!-- complete inertial system of the body -->
 <!-- FILE THAT INCLUDES GAZEBO OPTIONS AND MOTION CONTROLS-->
@@ -77,5 +77,5 @@
 <xacro:macro name = "body_link_macro">
    <inertial>
-   <origin rpy = "0 0 0" xyz = " 0 0 ${s1}"/>
+   <origin xyz = " 0 0 ${s1}" rpy = "0 0 0"/>
    <mass value = "${body_mass}"/>
    <inertia ixx ="${Ix_body}" ixy = "0.0" ixz ="0.0" iyy ="${Iy_body}" iyz = "0.0" izz= "${Iz_body}"/>
@@ -85,5 +85,5 @@
 <xacro:macro name = "wheel_link_macro">
    <inertial>
-   <origin rpy = " 1.570795 0 0" xyz = "0 0 0" />
+   <origin xyz = "0 0 0" rpy = " 1.570795 0 0"/>
    <mass value = "${wheel_mass}"/>
    <inertia ixx ="${Ix_wheel}" ixy="0.0" ixz="0.0" iyy="${Iy_wheel}" iyz ="0.0" izz="${Iz_wheel}"/>
@@ -93,16 +93,16 @@
 <xacro:macro name = "castor_link_macro">
    <inertial>
-   <origin rpy = "0 0 0" xyz = "0 0 0" />
+   <origin xyz = "0 0 0" rpy = "0 0 0"/>
    <mass value = "${castor_mass}"/>
    <inertia ixx = "${Ix_castor}" ixy= "0.0" ixz="0.0" iyy="${Iy_castor}" iyz="0.0" izz= "${Iz_castor}"/>
    </inertial>
 </xacro:macro>
+<!-- INERTFACE FOR COMTROLS -->
 <!-- FICTOUS LINK  -->
 <!-- DEFINING LINKS ANDS JOINTS -->
-<link name  = "base_footprint"></link>
+<link name  = "body_footprint"></link>
 <joint name = "body_link_joint" type = "fixed">
-   <parent link = "base_footprint"/>
+   <parent link = "body_footprint"/>
    <child link = "body_link"/>
-   <origin xyz= "0 0 0"/>
 </joint>
 <!-- BODY LINK OF ROBOT -->
@@ -110,13 +110,13 @@
    <visual>
       <geometry>
-         <box size = "${body_length} ${body_height} ${body_width}"/>
+         <box size = "${body_length} ${body_width} ${body_height}"/>
       </geometry>
-      <origin rpy = "0 0 0" xyz="0 0 ${s1}"/>
+      <origin xyz="0 0 ${s1}" rpy = "0 0 0"/>
    </visual>
    <collision>
       <geometry>
-         <box size = "${body_length} ${body_height} ${body_width}"/>
+         <box size = "${body_length} ${body_width} ${body_height}"/>
       </geometry>
-      <origin rpy = "0 0 0" xyz="0 0 ${s1}" />
+      <origin xyz="0 0 ${s1}" rpy = "0 0 0"/>
    </collision>
    <xacro:body_link_macro/>
@@ -127,5 +127,5 @@
    <child link = "wheel1_link"/>
    <origin xyz= " ${-s2} ${-s4} ${radius}" rpy="0 0 0"/>
-   <axis xyz= "0 0 1"/>
+   <axis xyz= "0 1 0"/>
    <limit effort = "100000" velocity= "10"/>
    <dynamics damping ="1.0" friction ="1.0"/>
@@ -150,5 +150,5 @@
    <child link = "wheel2_link"/>
    <origin xyz= " ${-s2} ${s4} ${radius}" rpy="0 0 0"/>
-   <axis xyz= "0 0 1"/>
+   <axis xyz= "0 1 0"/>
    <limit effort = "100000" velocity= "10"/>
    <dynamics damping ="1.0" friction ="1.0"/>

Commit message: latest

File: src/mobile_robot/model/robot.xacro (robot description, xacro)
@@ -7,8 +7,8 @@
 <xacro:property name = "body_length"
    value ="1.0"/>
+<xacro:property name = "body_height"
+   value ="0.30"/>
 <xacro:property name = "body_width"
-   value ="0.3"/>
-<xacro:property name = "body_height"
-   value ="0.6"/>
+   value ="0.60"/>
 <!-- WHEEL DIMENSIONS  AND CASTOR DIMENSIONS -->
 <!-- RADIUS -->
@@ -17,5 +17,5 @@
 <!-- WIDTH  WHEEL -->
 <xacro:property name ="width"
-   value ="0.1"/>
+   value ="0.10"/>
 <!-- other dimensions -->
 <xacro:property name = "s1"

Commit message: postioning error sorted

File: src/mobile_robot/model/robot.xacro (robot description, xacro)
@@ -77,5 +77,5 @@
 <xacro:macro name = "body_link_macro">
    <inertial>
-   <origin xyz = " 0 0 ${s1}" rpy = "0 0 0"/>
+   <origin xyz = " 0 0 0" rpy = "0 0 0"/>
    <mass value = "${body_mass}"/>
    <inertia ixx ="${Ix_body}" ixy = "0.0" ixz ="0.0" iyy ="${Iy_body}" iyz = "0.0" izz= "${Iz_body}"/>

Commit message: updates

File: src/mobile_robot/model/robot.xacro (robot description, xacro)
@@ -77,5 +77,5 @@
 <xacro:macro name = "body_link_macro">
    <inertial>
-   <origin xyz = " 0 0 0" rpy = "0 0 0"/>
+   <origin xyz = " 0 0 ${s1}" rpy = "0 0 0"/>
    <mass value = "${body_mass}"/>
    <inertia ixx ="${Ix_body}" ixy = "0.0" ixz ="0.0" iyy ="${Iy_body}" iyz = "0.0" izz= "${Iz_body}"/>

Commit message: updated

File: src/mobile_robot/model/robot.xacro (robot description, xacro)
@@ -126,5 +126,5 @@
    <parent link = "body_link"/>
    <child link = "wheel1_link"/>
-   <origin xyz= " ${-s2} ${-s4} ${radius}" rpy="0 0 0"/>
+   <origin xyz= " ${-s2} ${-s4} 0" rpy="0 0 0"/>
    <axis xyz= "0 1 0"/>
    <limit effort = "100000" velocity= "10"/>
@@ -149,5 +149,5 @@
    <parent link = "body_link"/>
    <child link = "wheel2_link"/>
-   <origin xyz= " ${-s2} ${s4} ${radius}" rpy="0 0 0"/>
+   <origin xyz= " ${-s2} ${s4} 0" rpy="0 0 0"/>
    <axis xyz= "0 1 0"/>
    <limit effort = "100000" velocity= "10"/>
@@ -170,8 +170,8 @@
 </link>
 <!-- CASTOR JOINT -->
-<joint name="caster_joint" type ="continuous">
+<joint name="caster_joint" type ="fixed">
    <parent link = "body_link"/>
    <child link = "caster_link"/>
-   <origin xyz= " ${body_length/2 - radius} 0 ${radius}" rpy="0 0 0"/>
+   <origin xyz= " ${body_length/2 - radius} 0 0" rpy="0 0 0"/>
    <axis xyz= "0 1 0"/>
    <limit effort = "100000" velocity= "10"/>

Commit message: robot postioning correct

File: src/mobile_robot/model/robot.xacro (robot description, xacro)
@@ -112,5 +112,5 @@
          <box size = "${body_length} ${body_width} ${body_height}"/>
       </geometry>
-      <origin xyz="0 0 ${s1}" rpy = "0 0 0"/>
+      <origin xyz="0 0 ${radius}" rpy = "0 0 0"/>
    </visual>
    <collision>
@@ -118,5 +118,5 @@
          <box size = "${body_length} ${body_width} ${body_height}"/>
       </geometry>
-      <origin xyz="0 0 ${s1}" rpy = "0 0 0"/>
+      <origin xyz="0 0 ${radius}" rpy = "0 0 0"/>
    </collision>
    <xacro:body_link_macro/>

Commit message: center of mass of body fixed

File: src/mobile_robot/model/robot.xacro (robot description, xacro)
@@ -77,5 +77,5 @@
 <xacro:macro name = "body_link_macro">
    <inertial>
-   <origin xyz = " 0 0 ${s1}" rpy = "0 0 0"/>
+   <origin xyz = " 0 0 ${radius}" rpy = "0 0 0"/>
    <mass value = "${body_mass}"/>
    <inertia ixx ="${Ix_body}" ixy = "0.0" ixz ="0.0" iyy ="${Iy_body}" iyz = "0.0" izz= "${Iz_body}"/>
@@ -93,5 +93,5 @@
 <xacro:macro name = "castor_link_macro">
    <inertial>
-   <origin xyz = "0 0 0" rpy = "0 0 0"/>
+   <origin xyz = "0 0 0" rpy = "1.57095 0 0"/>
    <mass value = "${castor_mass}"/>
    <inertia ixx = "${Ix_castor}" ixy= "0.0" ixz="0.0" iyy="${Iy_castor}" iyz="0.0" izz= "${Iz_castor}"/>
