Commit message: body everything correct now  and now the testing part

File: src/mobile_robot/model/robot.xacro (robot description, xacro)
@@ -170,8 +170,8 @@
 </link>
 <!-- CASTOR JOINT -->
-<joint name="caster_joint" type ="fixed">
+<joint name="caster_joint" type ="continuous">
    <parent link = "body_link"/>
    <child link = "caster_link"/>
-   <origin xyz= " ${body_length/2 - radius} 0 0" rpy="0 0 0"/>
+   <origin xyz= " ${body_length/2 - radius} 0 0" rpy="1.570795 0 0"/>
    <axis xyz= "0 1 0"/>
    <limit effort = "100000" velocity= "10"/>
@@ -183,5 +183,5 @@
          <sphere radius = "${radius}"/>
       </geometry>
-      <origin xyz = "0 0 0" rpy = "0 0 0"/>
+      <origin xyz = "0 0 0" rpy = "1.570795 0 0"/>
    </visual>
    <collision>
@@ -189,5 +189,5 @@
          <sphere radius = "${radius}"/>
       </geometry>
-      <origin xyz = "0 0 0" rpy = "0 0 0"/>
+      <origin xyz = "0 0 0" rpy = "1.570795 0 0"/>
    </collision>
    <xacro:castor_link_macro/>

Commit message: inertia corrected of thw body

File: src/mobile_robot/model/robot.xacro (robot description, xacro)
@@ -79,5 +79,5 @@
    <origin xyz = " 0 0 ${radius}" rpy = "0 0 0"/>
    <mass value = "${body_mass}"/>
-   <inertia ixx ="${Ix_body}" ixy = "0.0" ixz ="0.0" iyy ="${Iy_body}" iyz = "0.0" izz= "${Iz_body}"/>
+   <inertia ixx ="${Ix_body}" ixy = "0.0" ixz ="0.0" iyy ="${Iz_body}" iyz = "0.0" izz= "${Iy_body}"/>
    </inertial>
 </xacro:macro>

Commit message: lidar basicdimensions added

File: src/mobile_robot/model/robot.xacro (robot description, xacro)
@@ -193,3 +193,29 @@
    <xacro:castor_link_macro/>
 </link>
+<!-- LIDAR -->
+<joint name = "lidar_joint" type = "fixed">
+   <origin xyz="0 0 $(body_width+radius)" rpy="0 0 0"/>
+   <parent link="body_link"/>
+   <child link="lidar_link"/>
+   <axis xyz="0 1 0" rpy="0 0 0"/>
+</joint>
+<link name="lidar_link">
+   <visual>
+   <origin xyz="0 0 0.5" rpy="0 0 0"/>
+      <geometry>
+         <cylinder length ="0.1" radius="0.1"/>
+      </geometry>
+   </visual>
+   <collision name ="collision">
+      <origin xyz="0 0 0.05" rpy="0 0 0"/>
+      <geometry>
+         <cylinder length ="0.1" radius="0.1"/>
+      </geometry>
+   </collision>
+   <inertial>
+      <mass value="1e-6"/>
+      <origin xyz="0 0 0" rpy="0 0 0"/>
+      <inertia ixx="1e-6" ixy="0" ixz="0" iyy="1e-6" iyz="0" izz="1e-6"/>
+   </inertial>
+</link>
 </robot>

Commit message: LIDAR positioning corrected

File: src/mobile_robot/model/robot.xacro (robot description, xacro)
@@ -195,5 +195,5 @@
 <!-- LIDAR -->
 <joint name = "lidar_joint" type = "fixed">
-   <origin xyz="0 0 $(body_width+radius)" rpy="0 0 0"/>
+   <origin xyz="0 0 ${radius+body_height/2+0.05}" rpy="0 0 0"/>
    <parent link="body_link"/>
    <child link="lidar_link"/>
@@ -202,5 +202,5 @@
 <link name="lidar_link">
    <visual>
-   <origin xyz="0 0 0.5" rpy="0 0 0"/>
+   <origin xyz="0 0 0" rpy="0 0 0"/>
       <geometry>
          <cylinder length ="0.1" radius="0.1"/>
@@ -208,5 +208,5 @@
    </visual>
    <collision name ="collision">
-      <origin xyz="0 0 0.05" rpy="0 0 0"/>
+      <origin xyz="0 0 0" rpy="0 0 0"/>
       <geometry>
          <cylinder length ="0.1" radius="0.1"/>

Commit message: lidar positioning chnaged

File: src/mobile_robot/model/robot.xacro (robot description, xacro)
@@ -195,5 +195,5 @@
 <!-- LIDAR -->
 <joint name = "lidar_joint" type = "fixed">
-   <origin xyz="0 0 ${radius+body_height/2+0.05}" rpy="0 0 0"/>
+   <origin xyz="0 0 0.35" rpy="0 0 0"/>
    <parent link="body_link"/>
    <child link="lidar_link"/>

Commit message: wheel 3 added castor removed

File: src/mobile_robot/model/robot.xacro (robot description, xacro)
@@ -1,4 +1,4 @@
 <?xml version='1.0'?>
-<robot name = "castor_robot" xmlns:xacro="http://www.ros.org/wiki/xacro">
+<robot name = "diff_robot" xmlns:xacro="http://www.ros.org/wiki/xacro">
 <!-- define constants -->
 <xacro:property name = "ohm" value ="3.14159"/>
@@ -18,4 +18,6 @@
 <xacro:property name ="width"
    value ="0.10"/>
+<xacro:property name ="wheel_z_location"
+   value ="-0.1"/>
 <!-- other dimensions -->
 <xacro:property name = "s1"
@@ -35,7 +37,7 @@
 <xacro:property name = "wheel_link"
    value = "500.0"/>
-<!-- CASTOR LINK -->
+<!-- CASTOR LINK
 <xacro:property name = "castor_link"
-   value = "500.0"/>
+   value = "500.0"/> -->
 <!-- MASS -->
 <!-- BODY LINK MASS -->
@@ -45,7 +47,7 @@
 <xacro:property name = "wheel_mass"
    value = "${wheel_link*ohm*radius*radius*width}"/>
-<!-- CASTOR LINK MASS -->
+<!-- CASTOR LINK MASS
 <xacro:property name = "castor_mass"
-   value = "${castor_link*(4/3)*ohm*radius*radius*radius}"/>
+   value = "${castor_link*(4/3)*ohm*radius*radius*radius}"/> -->
 <!--MOMENT OF INERTIA -->
 <!-- BODY LINK MOMENT OF INERTIA -->
@@ -63,5 +65,5 @@
 <xacro:property name="Iz_wheel"
    value="${(1/12)*wheel_mass*(3*radius*radius + width*width)}"/>
-<!-- CASTOR LINK MOMENT OF INERTIA -->
+<!-- CASTOR LINK MOMENT OF INERTIA
 <xacro:property name = "Ix_castor"
    value = "${(2/5)*castor_mass*radius*radius}" />
@@ -69,9 +71,16 @@
    value = "${(2/5)*castor_mass*radius*radius}" />
 <xacro:property name = "Iz_castor"
-   value = "${(2/5)*castor_mass*radius*radius}" />
+   value = "${(2/5)*castor_mass*radius*radius}" /> -->
 <!-- complete inertial system of the body -->
 <!-- FILE THAT INCLUDES GAZEBO OPTIONS AND MOTION CONTROLS-->
 <xacro:include filename ="$(find mobile_robot)/model/robot.gazebo.xacro"/>
 <!-- THE BASIC COORDINATE SYSTEM IS CENTERED AT THE GEOMETRIC CENTER OF THE BODY LINK -->
+<!--dummy link for gazebo -->
+<link name="dummy">
+</link>
+<joint name="dummy_joint" type="fixed">
+   <parent link="dummy"/>
+   <child link="body_link"/>
+</joint>
 <!-- BODY LINK -->
 <xacro:macro name = "body_link_macro">
@@ -90,5 +99,5 @@
    </inertial>
 </xacro:macro>
-<!-- CASTOR LINK -->
+<!-- CASTOR LINK
 <xacro:macro name = "castor_link_macro">
    <inertial>
@@ -97,5 +106,5 @@
    <inertia ixx = "${Ix_castor}" ixy= "0.0" ixz="0.0" iyy="${Iy_castor}" iyz="0.0" izz= "${Iz_castor}"/>
    </inertial>
-</xacro:macro>
+</xacro:macro> -->
 <!-- INERTFACE FOR COMTROLS -->
 <!-- FICTOUS LINK  -->
@@ -169,5 +178,28 @@
    <xacro:wheel_link_macro/>
 </link>
-<!-- CASTOR JOINT -->
+<joint name="wheel3_joint" type ="continous">
+   <parent link="body_link"/>
+   <child link="wheel3_link"/>
+   <origin xyz="${s2} ${-s4} 0" rpy="0 0 0"/>
+   <axis xyz= "0 1 0"/>
+   <limit effort = "100000" velocity= "10"/>
+   <dynamics damping ="1.0" friction ="1.0"/>
+</joint>
+<link name = "wheel3_link"/>
+   <visual>
+      <geometry>
+         <cylinder length = "${width}" radius = "${radius}"/>
+      </geometry>
+      <origin xyz = "0 0 0" rpy = "1.570795 0 0"/>
+   </visual>
+   <collision>
+      <geometry>
+         <cylinder length = "${width}" radius = "${radius}"/>
+      </geometry>
+      <origin xyz = "0 0 0" rpy = "1.570795 0 0"/>
+   </collision>
+   <xacro:wheel_link_macro/>
+</link>
+<!-- CASTOR JOINT
 <joint name="caster_joint" type ="continuous">
    <parent link = "body_link"/>
@@ -192,5 +224,5 @@
    </collision>
    <xacro:castor_link_macro/>
-</link>
+</link>   -->
 <!-- LIDAR -->
 <joint name = "lidar_joint" type = "fixed">

Commit message: wheel 4 added

File: src/mobile_robot/model/robot.xacro (robot description, xacro)
@@ -201,4 +201,27 @@
    <xacro:wheel_link_macro/>
 </link>
+<joint name="wheel4_joint" type ="continous">
+   <parent link="body_link"/>
+   <child link="wheel3_link"/>
+   <origin xyz="${s2} ${s4} 0" rpy="0 0 0"/>
+   <axis xyz= "0 1 0"/>
+   <limit effort = "100000" velocity= "10"/>
+   <dynamics damping ="1.0" friction ="1.0"/>
+</joint>
+<link name = "wheel4_link"/>
+   <visual>
+      <geometry>
+         <cylinder length = "${width}" radius = "${radius}"/>
+      </geometry>
+      <origin xyz = "0 0 0" rpy = "1.570795 0 0"/>
+   </visual>
+   <collision>
+      <geometry>
+         <cylinder length = "${width}" radius = "${radius}"/>
+      </geometry>
+      <origin xyz = "0 0 0" rpy = "1.570795 0 0"/>
+   </collision>
+   <xacro:wheel_link_macro/>
+</link>
 <!-- CASTOR JOINT
 <joint name="caster_joint" type ="continuous">

Commit message: latest run

File: src/mobile_robot/model/robot.xacro (robot description, xacro)
@@ -163,20 +163,20 @@
    <dynamics damping ="1.0" friction ="1.0"/>
 </joint>
-<link name = "wheel2_link">
-   <visual>
-      <geometry>
-         <cylinder length = "${width}" radius = "${radius}"/>
-      </geometry>
-      <origin xyz = "0 0 0" rpy = "1.570795 0 0"/>
-   </visual>
-   <collision>
-      <geometry>
-         <cylinder length = "${width}" radius = "${radius}"/>
-      </geometry>
-      <origin xyz = "0 0 0" rpy = "1.570795 0 0"/>
-   </collision>
-   <xacro:wheel_link_macro/>
-</link>
-<joint name="wheel3_joint" type ="continous">
+<link name ="wheel2_link">
+   <visual>
+      <geometry>
+         <cylinder length = "${width}" radius = "${radius}"/>
+      </geometry>
+      <origin xyz = "0 0 0" rpy = "1.570795 0 0"/>
+   </visual>
+   <collision>
+      <geometry>
+         <cylinder length = "${width}" radius = "${radius}"/>
+      </geometry>
+      <origin xyz = "0 0 0" rpy = "1.570795 0 0"/>
+   </collision>
+   <xacro:wheel_link_macro/>
+</link>
+<joint name="wheel3_joint" type ="continuous">
    <parent link="body_link"/>
    <child link="wheel3_link"/>
@@ -186,39 +186,47 @@
    <dynamics damping ="1.0" friction ="1.0"/>
 </joint>
-<link name = "wheel3_link"/>
-   <visual>
-      <geometry>
-         <cylinder length = "${width}" radius = "${radius}"/>
-      </geometry>
-      <origin xyz = "0 0 0" rpy = "1.570795 0 0"/>
-   </visual>
-   <collision>
-      <geometry>
-         <cylinder length = "${width}" radius = "${radius}"/>
-      </geometry>
-      <origin xyz = "0 0 0" rpy = "1.570795 0 0"/>
-   </collision>
-   <xacro:wheel_link_macro/>
-</link>
-<joint name="wheel4_joint" type ="continous">
+<joint name="wheel3_joint" type="continuous">
    <parent link="body_link"/>
    <child link="wheel3_link"/>
+   <origin xyz="${s2} ${-s4} 0" rpy="0 0 0"/>
+   <axis xyz="0 1 0"/>
+   <limit effort="100000" velocity="10"/>
+   <dynamics damping="1.0" friction="1.0"/>
+</joint>
+<link name="wheel3_link">
+   <visual>
+      <geometry>
+         <cylinder length="${width}" radius="${radius}"/>
+      </geometry>
+      <origin xyz="0 0 0" rpy="1.570795 0 0"/>
+   </visual>
+   <collision>
+      <geometry>
+         <cylinder length="${width}" radius="${radius}"/>
+      </geometry>
+      <origin xyz="0 0 0" rpy="1.570795 0 0"/>
+   </collision>
+   <xacro:wheel_link_macro/>
+</link>
+<joint name="wheel4_joint" type="continuous">
+   <parent link="body_link"/>
+   <child link="wheel4_link"/>
    <origin xyz="${s2} ${s4} 0" rpy="0 0 0"/>
-   <axis xyz= "0 1 0"/>
-   <limit effort = "100000" velocity= "10"/>
-   <dynamics damping ="1.0" friction ="1.0"/>
-</joint>
-<link name = "wheel4_link"/>
-   <visual>
-      <geometry>
-         <cylinder length = "${width}" radius = "${radius}"/>
-      </geometry>
-      <origin xyz = "0 0 0" rpy = "1.570795 0 0"/>
-   </visual>
-   <collision>
-      <geometry>
-         <cylinder length = "${width}" radius = "${radius}"/>
-      </geometry>
-      <origin xyz = "0 0 0" rpy = "1.570795 0 0"/>
+   <axis xyz="0 1 0"/>
+   <limit effort="100000" velocity="10"/>
+   <dynamics damping="1.0" friction="1.0"/>
+</joint>
+<link name="wheel4_link">
+   <visual>
+      <geometry>
+         <cylinder length="${width}" radius="${radius}"/>
+      </geometry>
+      <origin xyz="0 0 0" rpy="1.570795 0 0"/>
+   </visual>
+   <collision>
+      <geometry>
+         <cylinder length="${width}" radius="${radius}"/>
+      </geometry>
+      <origin xyz="0 0 0" rpy="1.570795 0 0"/>
    </collision>
    <xacro:wheel_link_macro/>

Commit message: updated

File: src/mobile_robot/model/robot.xacro (robot description, xacro)
@@ -1,4 +1,4 @@
 <?xml version='1.0'?>
-<robot name = "diff_robot" xmlns:xacro="http://www.ros.org/wiki/xacro">
+<robot name = "castor_robot" xmlns:xacro="http://www.ros.org/wiki/xacro">
 <!-- define constants -->
 <xacro:property name = "ohm" value ="3.14159"/>
@@ -178,12 +178,4 @@
    <xacro:wheel_link_macro/>
 </link>
-<joint name="wheel3_joint" type ="continuous">
-   <parent link="body_link"/>
-   <child link="wheel3_link"/>
-   <origin xyz="${s2} ${-s4} 0" rpy="0 0 0"/>
-   <axis xyz= "0 1 0"/>
-   <limit effort = "100000" velocity= "10"/>
-   <dynamics damping ="1.0" friction ="1.0"/>
-</joint>
 <joint name="wheel3_joint" type="continuous">
    <parent link="body_link"/>

Commit message: latest design

File: src/mobile_robot/model/robot.xacro (robot description, xacro)
@@ -76,5 +76,5 @@
 <xacro:include filename ="$(find mobile_robot)/model/robot.gazebo.xacro"/>
 <!-- THE BASIC COORDINATE SYSTEM IS CENTERED AT THE GEOMETRIC CENTER OF THE BODY LINK -->
-<!--dummy link for gazebo -->
+<!-- dummy link for gazebo
 <link name="dummy">
 </link>
@@ -82,5 +82,5 @@
    <parent link="dummy"/>
    <child link="body_link"/>
-</joint>
+</joint> -->
 <!-- BODY LINK -->
 <xacro:macro name = "body_link_macro">
@@ -94,5 +94,5 @@
 <xacro:macro name = "wheel_link_macro">
    <inertial>
-   <origin xyz = "0 0 0" rpy = " 1.570795 0 0"/>
+   <origin xyz = "0 0 0" rpy = "0 0 0"/>
    <mass value = "${wheel_mass}"/>
    <inertia ixx ="${Ix_wheel}" ixy="0.0" ixz="0.0" iyy="${Iy_wheel}" iyz ="0.0" izz="${Iz_wheel}"/>
